File: kleingorium_20250427163006-backups/kleingorium_old.kicad_pcb (KiCad board)
At the start: 2 copper layers, 100 x 100 mm, 42 parts, among them J1 4017 Pins, J10 VCC, J11 GND, J12 4046 Comp In, J2 4040 Output, J3 4040 Input, J4 4046 Out, J5 4046 Comp, J6 Select, J7 Output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

Commit message: renaming
Parts:
- removed C10: 10uF, Capacitor_THT:CP_Radial_D5.0mm_P2.50mm
- removed C11, C12, C13, C14, C15: 100nF, Capacitor_THT:C_Disc_D3.0mm_W1.6mm_P2.50mm
- removed SW3: Chain, Button_Switch_THT:SW_E-Switch_EG1271_SPDT
- added C4: 100nF, Capacitor_THT:C_Disc_D3.0mm_W1.6mm_P2.50mm, F.Cu at (101.4, 106.8)
- added C5: 100nF, Capacitor_THT:C_Disc_D3.0mm_W1.6mm_P2.50mm, F.Cu at (180.0, 99.8)
- added C6: 100nF, Capacitor_THT:C_Disc_D3.0mm_W1.6mm_P2.50mm, F.Cu at (175.0, 123.5)
- added C7: 100nF, Capacitor_THT:C_Disc_D3.0mm_W1.6mm_P2.50mm, F.Cu at (138.5, 107.4)
- added C8: 100nF, Capacitor_THT:C_Disc_D3.0mm_W1.6mm_P2.50mm, F.Cu at (138.5, 91.4)
- added C9: 10uF, Capacitor_THT:CP_Radial_D5.0mm_P2.50mm, F.Cu at (94.2, 113.5)
- Q1: footprint Package_TO_SOT_THT:TO-92_Inline_Wide -> Package_TO_SOT_THT:TO-92_Inline
- U1: value 4046 -> CD4053B
- U2: value 4017 -> 4046
- U3: value CD4053B -> 4017
- moved U3 68.0 mm to (197.6, 118.5), turned to -90 degrees
- moved U4 47.6 mm to (201.9, 94.7), turned to -90 degrees
- moved R8 42.5 mm to (204.0, 129.1), turned to 90 degrees
- moved R9 42.2 mm to (207.0, 129.1), turned to 90 degrees
- moved R3 40.5 mm to (160.0, 113.5)
- moved R4 40.1 mm to (157.0, 113.5)
- moved U5 34.8 mm to (159.6, 86.2), turned to -90 degrees
- moved U1 29.7 mm to (124.3, 101.7), turned to -90 degrees
- moved U2 29.3 mm to (161.4, 102.2), turned to -90 degrees
- moved C1 27.4 mm to (151.0, 99.5), turned to 180 degrees
- moved J2 26.7 mm to (177.8, 108.9)
- moved C2 19.9 mm to (147.8, 113.0), turned to 0 degrees
- moved J1 19.6 mm to (172.8, 143.0)
- moved J9 16.0 mm to (138.7, 114.5)
- moved R6 15.0 mm to (157.5, 139.5)
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Connections:
- C1 pad 1: Net-(U1-C1) -> Net-(U2-C1)
- C1 pad 2: Net-(U1-C2) -> Net-(U2-C2)
- C2 pad 1: Net-(U1-SigIn) -> Net-(U2-SigIn)
- J7 pad 2: Net-(J7-Pin_2) -> /4053/C
- Q1 pad 3: /4066/Ben -> /4066/Cen
- R1 pad 1: Net-(U3-INH) -> Net-(U1-INH)
- R11 pad 2: /4066/Ben -> /4066/Cen
- R3 pad 1: Net-(U1-Inh) -> Net-(U2-Inh)
- R4 pad 1: Net-(U1-R1) -> Net-(U2-R1)
- R5 pad 1: Net-(U1-PC2) -> Net-(U2-PC2)
- R5 pad 2: Net-(U1-VCOin) -> Net-(U2-VCOin)
- R5 pad 3: Net-(U1-VCOin) -> Net-(U2-VCOin)
- R6 pad 1: Net-(U1-VCOin) -> Net-(U2-VCOin)
- U1 pad 1: unconnected-(U1-PCP-Pad1) -> /4053/B1
- U1 pad 10: unconnected-(U1-SFout-Pad10) -> /4053/Select
- U1 pad 11: Net-(U1-R1) -> /4053/Select
- U1 pad 12: unconnected-(U1-R2-Pad12) -> /4017/Clock
- U1 pad 13: Net-(U1-PC2) -> /4046/SigIn
- U1 pad 14: Net-(U1-SigIn) -> /4053/A
- U1 pad 15: unconnected-(U1-ZOUT-Pad15) -> /4053/B
- U1 pad 2: unconnected-(U1-PC1-Pad2) -> /4046/SigIn
- U1 pad 3: /4046/Comp -> /4040/Q2
- U1 pad 4: /4040/Clock -> /4053/C
- U1 pad 5: Net-(U1-Inh) -> /4040/Clock
- U1 pad 6: Net-(U1-C1) -> Net-(U1-INH)
- U1 pad 7: Net-(U1-C2) -> GND
- U1 pad 9: Net-(U1-VCOin) -> /4053/Select
- U2 pad 1: /4017/Q5 -> unconnected-(U2-PCP-Pad1)
- U2 pad 10: /4017/Q4 -> unconnected-(U2-SFout-Pad10)
- U2 pad 11: /4017/Q9 -> Net-(U2-R1)
- U2 pad 12: /4017/Q10 -> unconnected-(U2-R2-Pad12)
- U2 pad 13: /4017/ClockEnable -> Net-(U2-PC2)
- U2 pad 14: /4017/Clock -> Net-(U2-SigIn)
- U2 pad 15: /4017/Reset -> unconnected-(U2-ZOUT-Pad15)
- U2 pad 2: /4017/Q1 -> unconnected-(U2-PC1-Pad2)
- U2 pad 3: /4017/Q0 -> /4046/Comp
- U2 pad 4: /4017/Q2 -> /4040/Clock
- U2 pad 5: /4017/Q6 -> Net-(U2-Inh)
- U2 pad 6: /4017/Q7 -> Net-(U2-C1)
- U2 pad 7: /4017/Q3 -> Net-(U2-C2)
- U2 pad 9: /4017/Q8 -> Net-(U2-VCOin)
- U3 pad 1: /4053/B1 -> /4017/Q5
- U3 pad 10: /4053/Select -> /4017/Q4
- U3 pad 11: /4053/Select -> /4017/Q9
- U3 pad 12: /4017/Clock -> /4017/Q10
- U3 pad 13: /4046/SigIn -> /4017/ClockEnable
- U3 pad 14: /4053/A -> /4017/Clock
- U3 pad 15: /4053/B -> /4017/Reset
- U3 pad 2: /4046/SigIn -> /4017/Q1
- U3 pad 3: /4040/Q2 -> /4017/Q0
- U3 pad 4: /4053/C -> /4017/Q2
- U3 pad 5: /4040/Clock -> /4017/Q6
- U3 pad 6: Net-(U3-INH) -> /4017/Q7
- U3 pad 7: GND -> /4017/Q3
- U3 pad 9: /4053/Select -> /4017/Q8
- U5 pad 1: /4053/B1 -> /4066/A1
- U5 pad 10: /4066/D2 -> /4017/Clock
- U5 pad 11: /4066/D1 -> /4040/Clock
- U5 pad 12: /4066/Den -> /4053/Select
- U5 pad 13: /4053/Select -> /4066/Aen
- U5 pad 2: /4040/Q2 -> /4066/A2
- U5 pad 3: /4017/Clock -> /4066/B2
- U5 pad 4: /4040/Clock -> /4066/B1
- U5 pad 8: /4066/C1 -> /4053/B1
- U5 pad 9: /4066/C2 -> /4040/Q2
Routing:
- net VCC: track 0.00 -> 240.4 mm, vias 0 -> 3
- net /4053/Select: track 0.00 -> 116.3 mm, vias 0 -> 2
- net /4017/Reset: track 0.00 -> 109.8 mm
- net /4040/Clock: track 5.22 -> 113.7 mm, vias 0 -> 2
- net /4017/Clock: track 0.00 -> 103.2 mm, vias 0 -> 1
- net /4053/B1: track 0.00 -> 89.8 mm
- net /4066/Cen: track 0.00 -> 73.9 mm, vias 0 -> 1
- net /4040/Q2: track 24.0 -> 91.6 mm
- net /4017/Q0: track 19.7 -> 86.0 mm, vias 0 -> 1
- net /4046/Comp: track 0.00 -> 57.7 mm, vias 0 -> 1
- net Net-(U2-VCOin): track 0.00 -> 52.0 mm
- net /4046/SigIn: track 0.00 -> 48.6 mm
- net /4053/A: track 0.00 -> 37.1 mm
- net /4053/C: track 0.00 -> 35.5 mm
- net Net-(U2-PC2): track 0.00 -> 35.5 mm
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- removed copper zone on F.Cu, net VCC
Other:
- board size 100 x 100 mm -> 126.5 x 72 mm
- board text added: "4 0 5 3"
- board text added: "4017"
- board text added: "4017 Feedback"
- board text added: "4046 CompIn"
- board text added: "Comp"
- board text added: "CompIn"
- board text removed: "4 0 1 7"
- board text removed: "4017 Fdbk"
- board text removed: "4046 CmpIn"
- board text removed: "4053"
- board text removed: "Chain"
- board text removed: "Cmp"
- board text removed: "CmpIn"
