File: kleingorium.kicad_pcb (KiCad board)
At the start: 2 copper layers, 100 x 100 mm, 83 parts, among them J1 4017 Pins, J10 VCC, J11 GND, J12 4046 Comp In, J13 Select, J14 Input, J15 4046 SigIn, J16 4046 Comp, J17 Output, J18 4046 Comp In, J19 4046 Out, J2 4040 Output, J20 4040 Input, J21 4040 Output, J22 4017 Pins, J23 VCC, J24 GND, J3 4040 Input, J4 4046 Out, J5 4046 Comp, J6 Select, J7 Output, J8 Input, J9 4046 SigIn, Q1 2N3904, Q2 2N3904, SW1 4017 Feedback, SW2 4046 CompIn, SW3 Chain, SW4 4017 Feedback, SW5 4046 CompIn, U1 4046, U12 4040, U13 CD4053B, U14 4017, U15 4046, U2 4017, U3 CD4053B, U4 4040, U5 CD4066BE

Commit message: remove pull down resistor, change pull up from 10k to 2.2k
Parts:
- removed R15, R16: 10k, Resistor_THT:R_Axial_DIN0207_L6.3mm_D2.5mm_P10.16mm_Horizontal
- R11, R14: value 10k -> 2.2k
Routing:
- net /4066/Aen: track 63.5 -> 54.4 mm
- net /4066/Den: track 70.8 -> 64.7 mm
- net /4053 2/Select: track 182.7 -> 177.4 mm
- net Net-(C9-Pad2): track 8.13 -> 7.29 mm
- net Net-(C3-Pad2): track 8.33 -> 7.48 mm
