File: 4040.kicad_sch (KiCad schematic)
At the start: 2 parts, among them U4 4040

Commit message: v2 initial commit
Parts:
- renumbered U4 to U3
Changed lines of the file:
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@@
 		(dnp no)
 		(fields_autoplaced yes)
-		(property "Reference" "#PWR0105"
+		(property "Reference" "#PWR012"
 			(at 133.35 53.34 0)
 			(effects
@@
 		(instances
 			(project "kleingorium"
-				(path "/01c1f2c1-4d06-4880-847a-9ab55552e3fd/52b875be-0119-4d8e-9a5f-5c83f9081af4"
-					(reference "#PWR0105")
-					(unit 1)
-				)
-				(path "/01c1f2c1-4d06-4880-847a-9ab55552e3fd/cd1975a8-69a9-42c9-8d5e-87a03483f676"
-					(reference "#PWR059")
+				(path "/01c1f2c1-4d06-4880-847a-9ab55552e3fd/ad1f1d92-237d-4bc3-883c-2ce266dd223f/6ef5057d-5d74-4c3b-b2d1-eb9e2a0d3641"
+					(reference "#PWR012")
 					(unit 1)
 				)
@@
 		(dnp no)
 		(fields_autoplaced yes)
-		(property "Reference" "#PWR019"
+		(property "Reference" "#PWR011"
 			(at 116.84 99.06 0)
 			(effects
@@
 		(instances
 			(project "kleingorium"
-				(path "/01c1f2c1-4d06-4880-847a-9ab55552e3fd/52b875be-0119-4d8e-9a5f-5c83f9081af4"
-					(reference "#PWR019")
-					(unit 1)
-				)
-				(path "/01c1f2c1-4d06-4880-847a-9ab55552e3fd/cd1975a8-69a9-42c9-8d5e-87a03483f676"
-					(reference "#PWR048")
+				(path "/01c1f2c1-4d06-4880-847a-9ab55552e3fd/ad1f1d92-237d-4bc3-883c-2ce266dd223f/6ef5057d-5d74-4c3b-b2d1-eb9e2a0d3641"
+					(reference "#PWR011")
 					(unit 1)
 				)
@@
 		(dnp no)
 		(fields_autoplaced yes)
-		(property "Reference" "#PWR0106"
+		(property "Reference" "#PWR013"
 			(at 133.35 99.06 0)
 			(effects
@@
 		(instances
 			(project "kleingorium"
-				(path "/01c1f2c1-4d06-4880-847a-9ab55552e3fd/52b875be-0119-4d8e-9a5f-5c83f9081af4"
-					(reference "#PWR0106")
-					(unit 1)
-				)
-				(path "/01c1f2c1-4d06-4880-847a-9ab55552e3fd/cd1975a8-69a9-42c9-8d5e-87a03483f676"
-					(reference "#PWR060")
+				(path "/01c1f2c1-4d06-4880-847a-9ab55552e3fd/ad1f1d92-237d-4bc3-883c-2ce266dd223f/6ef5057d-5d74-4c3b-b2d1-eb9e2a0d3641"
+					(reference "#PWR013")
 					(unit 1)
 				)
@@
 		(dnp no)
 		(fields_autoplaced yes)
-		(property "Reference" "U4"
+		(property "Reference" "U3"
 			(at 135.4933 49.53 0)
 			(effects
@@
 		(instances
 			(project "kleingorium"
-				(path "/01c1f2c1-4d06-4880-847a-9ab55552e3fd/52b875be-0119-4d8e-9a5f-5c83f9081af4"
-					(reference "U4")
-					(unit 1)
-				)
-				(path "/01c1f2c1-4d06-4880-847a-9ab55552e3fd/cd1975a8-69a9-42c9-8d5e-87a03483f676"
-					(reference "U12")
+				(path "/01c1f2c1-4d06-4880-847a-9ab55552e3fd/ad1f1d92-237d-4bc3-883c-2ce266dd223f/6ef5057d-5d74-4c3b-b2d1-eb9e2a0d3641"
+					(reference "U3")
 					(unit 1)
 				)
@@
 		(instances
 			(project "kleingorium"
-				(path "/01c1f2c1-4d06-4880-847a-9ab55552e3fd/52b875be-0119-4d8e-9a5f-5c83f9081af4"
+				(path "/01c1f2c1-4d06-4880-847a-9ab55552e3fd/ad1f1d92-237d-4bc3-883c-2ce266dd223f/6ef5057d-5d74-4c3b-b2d1-eb9e2a0d3641"
 					(reference "R7")
 					(unit 1)
 				)
-				(path "/01c1f2c1-4d06-4880-847a-9ab55552e3fd/cd1975a8-69a9-42c9-8d5e-87a03483f676"
-					(reference "R27")
-					(unit 1)
-				)
