File: 4040.kicad_sch (KiCad schematic)
At the start: 2 parts, among them U3 4040

Commit message: wip symmetric layout
Parts:
- renumbered R12 to R23, U3 to U7
Changed lines of the file:
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@@
 		(dnp no)
 		(fields_autoplaced yes)
-		(property "Reference" "#PWR021"
+		(property "Reference" "#PWR040"
 			(at 133.35 53.34 0)
 			(effects
@@
 		(instances
 			(project "kleingorium"
-				(path "/01c1f2c1-4d06-4880-847a-9ab55552e3fd/ad1f1d92-237d-4bc3-883c-2ce266dd223f/52c73a40-bd38-49e3-8e94-4048d0c90ea6"
-					(reference "#PWR043")
-					(unit 1)
-				)
-				(path "/01c1f2c1-4d06-4880-847a-9ab55552e3fd/ad1f1d92-237d-4bc3-883c-2ce266dd223f/6ef5057d-5d74-4c3b-b2d1-eb9e2a0d3641"
-					(reference "#PWR021")
+				(path "/01c1f2c1-4d06-4880-847a-9ab55552e3fd/ad1f1d92-237d-4bc3-883c-2ce266dd223f/4b203833-f0af-4e88-a9fb-191df5175df3/56f505af-8cb7-4073-afe4-6d98c7fe6832"
+					(reference "#PWR011")
+					(unit 1)
+				)
+				(path "/01c1f2c1-4d06-4880-847a-9ab55552e3fd/ad1f1d92-237d-4bc3-883c-2ce266dd223f/e00ebc01-440e-4477-8d51-aed2c51c95ea/56f505af-8cb7-4073-afe4-6d98c7fe6832"
+					(reference "#PWR040")
 					(unit 1)
 				)
@@
 		(dnp no)
 		(fields_autoplaced yes)
-		(property "Reference" "#PWR020"
+		(property "Reference" "#PWR039"
 			(at 116.84 99.06 0)
 			(effects
@@
 		(instances
 			(project "kleingorium"
-				(path "/01c1f2c1-4d06-4880-847a-9ab55552e3fd/ad1f1d92-237d-4bc3-883c-2ce266dd223f/52c73a40-bd38-49e3-8e94-4048d0c90ea6"
-					(reference "#PWR042")
-					(unit 1)
-				)
-				(path "/01c1f2c1-4d06-4880-847a-9ab55552e3fd/ad1f1d92-237d-4bc3-883c-2ce266dd223f/6ef5057d-5d74-4c3b-b2d1-eb9e2a0d3641"
-					(reference "#PWR020")
+				(path "/01c1f2c1-4d06-4880-847a-9ab55552e3fd/ad1f1d92-237d-4bc3-883c-2ce266dd223f/4b203833-f0af-4e88-a9fb-191df5175df3/56f505af-8cb7-4073-afe4-6d98c7fe6832"
+					(reference "#PWR010")
+					(unit 1)
+				)
+				(path "/01c1f2c1-4d06-4880-847a-9ab55552e3fd/ad1f1d92-237d-4bc3-883c-2ce266dd223f/e00ebc01-440e-4477-8d51-aed2c51c95ea/56f505af-8cb7-4073-afe4-6d98c7fe6832"
+					(reference "#PWR039")
 					(unit 1)
 				)
@@
 		(dnp no)
 		(fields_autoplaced yes)
-		(property "Reference" "#PWR022"
+		(property "Reference" "#PWR041"
 			(at 133.35 99.06 0)
 			(effects
@@
 		(instances
 			(project "kleingorium"
-				(path "/01c1f2c1-4d06-4880-847a-9ab55552e3fd/ad1f1d92-237d-4bc3-883c-2ce266dd223f/52c73a40-bd38-49e3-8e94-4048d0c90ea6"
-					(reference "#PWR044")
-					(unit 1)
-				)
-				(path "/01c1f2c1-4d06-4880-847a-9ab55552e3fd/ad1f1d92-237d-4bc3-883c-2ce266dd223f/6ef5057d-5d74-4c3b-b2d1-eb9e2a0d3641"
-					(reference "#PWR022")
+				(path "/01c1f2c1-4d06-4880-847a-9ab55552e3fd/ad1f1d92-237d-4bc3-883c-2ce266dd223f/4b203833-f0af-4e88-a9fb-191df5175df3/56f505af-8cb7-4073-afe4-6d98c7fe6832"
+					(reference "#PWR012")
+					(unit 1)
+				)
+				(path "/01c1f2c1-4d06-4880-847a-9ab55552e3fd/ad1f1d92-237d-4bc3-883c-2ce266dd223f/e00ebc01-440e-4477-8d51-aed2c51c95ea/56f505af-8cb7-4073-afe4-6d98c7fe6832"
+					(reference "#PWR041")
 					(unit 1)
 				)
@@
 		(dnp no)
 		(fields_autoplaced yes)
-		(property "Reference" "U3"
+		(property "Reference" "U7"
 			(at 135.4933 49.53 0)
 			(effects
@@
 		(instances
 			(project "kleingorium"
-				(path "/01c1f2c1-4d06-4880-847a-9ab55552e3fd/ad1f1d92-237d-4bc3-883c-2ce266dd223f/52c73a40-bd38-49e3-8e94-4048d0c90ea6"
+				(path "/01c1f2c1-4d06-4880-847a-9ab55552e3fd/ad1f1d92-237d-4bc3-883c-2ce266dd223f/4b203833-f0af-4e88-a9fb-191df5175df3/56f505af-8cb7-4073-afe4-6d98c7fe6832"
+					(reference "U2")
+					(unit 1)
+				)
+				(path "/01c1f2c1-4d06-4880-847a-9ab55552e3fd/ad1f1d92-237d-4bc3-883c-2ce266dd223f/e00ebc01-440e-4477-8d51-aed2c51c95ea/56f505af-8cb7-4073-afe4-6d98c7fe6832"
 					(reference "U7")
-					(unit 1)
-				)
-				(path "/01c1f2c1-4d06-4880-847a-9ab55552e3fd/ad1f1d92-237d-4bc3-883c-2ce266dd223f/6ef5057d-5d74-4c3b-b2d1-eb9e2a0d3641"
-					(reference "U3")
 					(unit 1)
 				)
@@
 		(dnp no)
 		(fields_autoplaced yes)
-		(property "Reference" "R12"
+		(property "Reference" "R23"
 			(at 119.38 74.9299 0)
 			(effects
@@
 		(instances
 			(project "kleingorium"
-				(path "/01c1f2c1-4d06-4880-847a-9ab55552e3fd/ad1f1d92-237d-4bc3-883c-2ce266dd223f/52c73a40-bd38-49e3-8e94-4048d0c90ea6"
-					(reference "R25")
-					(unit 1)
-				)
-				(path "/01c1f2c1-4d06-4880-847a-9ab55552e3fd/ad1f1d92-237d-4bc3-883c-2ce266dd223f/6ef5057d-5d74-4c3b-b2d1-eb9e2a0d3641"
-					(reference "R12")
-					(unit 1)
-				)
+				(path "/01c1f2c1-4d06-4880-847a-9ab55552e3fd/ad1f1d92-237d-4bc3-883c-2ce266dd223f/4b203833-f0af-4e88-a9fb-191df5175df3/56f505af-8cb7-4073-afe4-6d98c7fe6832"
+					(reference "R5")
+					(unit 1)
+				)
+				(path "/01c1f2c1-4d06-4880-847a-9ab55552e3fd/ad1f1d92-237d-4bc3-883c-2ce266dd223f/e00ebc01-440e-4477-8d51-aed2c51c95ea/56f505af-8cb7-4073-afe4-6d98c7fe6832"
+					(reference "R23")
+					(unit 1)
+				)
