File: 4046.kicad_sch (KiCad schematic)
At the start: 8 parts, among them U1 4046

Commit message: schematic doubling without pcb placing
Parts:
- renumbered C1 to C
Changed lines of the file:
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@@
+					(unit 1)
+				)
+				(path "/01c1f2c1-4d06-4880-847a-9ab55552e3fd/ec892350-7ee5-4574-b787-aa0418288502"
+					(reference "C7")
 					(unit 1)
 				)
@@
 		(dnp no)
 		(fields_autoplaced yes)
-		(property "Reference" "#PWR015"
+		(property "Reference" "#PWR"
 			(at 152.4 50.8 0)
 			(effects
@@
 		)
 		(instances
-			(project ""
-				(path "/01c1f2c1-4d06-4880-847a-9ab55552e3fd/79441be6-e853-4219-9c9d-5fa446c925d2"
-					(reference "#PWR015")
+			(project "kleingorium"
+				(path "/01c1f2c1-4d06-4880-847a-9ab55552e3fd/ec892350-7ee5-4574-b787-aa0418288502"
+					(reference "#PWR067")
 					(unit 1)
 				)
@@
 					(unit 1)
 				)
+				(path "/01c1f2c1-4d06-4880-847a-9ab55552e3fd/ec892350-7ee5-4574-b787-aa0418288502"
+					(reference "U15")
+					(unit 1)
+				)
 			)
 		)
@@
 					(unit 1)
 				)
+				(path "/01c1f2c1-4d06-4880-847a-9ab55552e3fd/ec892350-7ee5-4574-b787-aa0418288502"
+					(reference "R34")
+					(unit 1)
+				)
 			)
 		)
@@
 					(unit 1)
 				)
+				(path "/01c1f2c1-4d06-4880-847a-9ab55552e3fd/ec892350-7ee5-4574-b787-aa0418288502"
+					(reference "#PWR051")
+					(unit 1)
+				)
 			)
 		)
@@
 					(unit 1)
 				)
+				(path "/01c1f2c1-4d06-4880-847a-9ab55552e3fd/ec892350-7ee5-4574-b787-aa0418288502"
+					(reference "R33")
+					(unit 1)
+				)
 			)
 		)
@@
 					(unit 1)
 				)
+				(path "/01c1f2c1-4d06-4880-847a-9ab55552e3fd/ec892350-7ee5-4574-b787-aa0418288502"
+					(reference "#PWR069")
+					(unit 1)
+				)
 			)
 		)
@@
 					(unit 1)
 				)
+				(path "/01c1f2c1-4d06-4880-847a-9ab55552e3fd/ec892350-7ee5-4574-b787-aa0418288502"
+					(reference "R30")
+					(unit 1)
+				)
 			)
 		)
@@
 					(unit 1)
 				)
+				(path "/01c1f2c1-4d06-4880-847a-9ab55552e3fd/ec892350-7ee5-4574-b787-aa0418288502"
+					(reference "#PWR068")
+					(unit 1)
+				)
 			)
 		)
@@
 					(unit 1)
 				)
+				(path "/01c1f2c1-4d06-4880-847a-9ab55552e3fd/ec892350-7ee5-4574-b787-aa0418288502"
+					(reference "R32")
+					(unit 1)
+				)
 			)
 		)
@@
 					(unit 1)
 				)
+				(path "/01c1f2c1-4d06-4880-847a-9ab55552e3fd/ec892350-7ee5-4574-b787-aa0418288502"
+					(reference "C9")
+					(unit 1)
+				)
 			)
 		)
@@
 					(unit 1)
 				)
+				(path "/01c1f2c1-4d06-4880-847a-9ab55552e3fd/ec892350-7ee5-4574-b787-aa0418288502"
+					(reference "#PWR064")
+					(unit 1)
+				)
 			)
 		)
@@
 		(on_board yes)
 		(dnp no)
-		(property "Reference" "C1"
+		(property "Reference" "C"
 			(at 127 67.31 0)
 			(effects
@@
 		)
 		(instances
-			(project ""
-				(path "/01c1f2c1-4d06-4880-847a-9ab55552e3fd/79441be6-e853-4219-9c9d-5fa446c925d2"
-					(reference "C1")
-					(unit 1)
-				)
+			(project "kleingorium"
+				(path "/01c1f2c1-4d06-4880-847a-9ab55552e3fd/ec892350-7ee5-4574-b787-aa0418288502"
+					(reference "C8")
+					(unit 1)
+				)

Commit message: pcb placing doubling without routing
Parts:
- renumbered C to C1
Changed lines of the file:
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@@
 		(dnp no)
 		(fields_autoplaced yes)
-		(property "Reference" "#PWR"
+		(property "Reference" "#PWR0101"
 			(at 152.4 50.8 0)
 			(effects
@@
 		(instances
 			(project "kleingorium"
+				(path "/01c1f2c1-4d06-4880-847a-9ab55552e3fd/79441be6-e853-4219-9c9d-5fa446c925d2"
+					(reference "#PWR0101")
+					(unit 1)
+				)
 				(path "/01c1f2c1-4d06-4880-847a-9ab55552e3fd/ec892350-7ee5-4574-b787-aa0418288502"
 					(reference "#PWR067")
@@
 		(on_board yes)
 		(dnp no)
-		(property "Reference" "C"
+		(property "Reference" "C1"
 			(at 127 67.31 0)
 			(effects
@@
 		(instances
 			(project "kleingorium"
+				(path "/01c1f2c1-4d06-4880-847a-9ab55552e3fd/79441be6-e853-4219-9c9d-5fa446c925d2"
+					(reference "C1")
+					(unit 1)
+				)
 				(path "/01c1f2c1-4d06-4880-847a-9ab55552e3fd/ec892350-7ee5-4574-b787-aa0418288502"
 					(reference "C8")

Commit message: fix errors with 4066 and Select
Parts:
- C2: footprint Capacitor_THT:C_Disc_D3.0mm_W1.6mm_P2.50mm -> Capacitor_THT:C_Disc_D4.3mm_W1.9mm_P5.00mm
- C3: footprint Capacitor_THT:C_Disc_D3.0mm_W1.6mm_P2.50mm -> Capacitor_THT:C_Disc_D5.0mm_W2.5mm_P5.00mm
Changed lines of the file:
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@@
 			)
 		)
-		(property "Footprint" "Capacitor_THT:C_Disc_D3.0mm_W1.6mm_P2.50mm"
+		(property "Footprint" "Capacitor_THT:C_Disc_D4.3mm_W1.9mm_P5.00mm"
 			(at 119.38 63.1952 0)
 			(effects
@@
 			)
 		)
-		(property "Footprint" "Capacitor_THT:C_Disc_D3.0mm_W1.6mm_P2.50mm"
+		(property "Footprint" "Capacitor_THT:C_Disc_D5.0mm_W2.5mm_P5.00mm"
 			(at 173.0248 85.09 0)
 			(effects

Commit message: change potentiometer legs R5 and R33
Connections:
- net at U1.13 (PC2): now also R5.3; no longer R5.1
- net at R5.2, R6.1, U1.9 (VCOin): now also R5.1; no longer R5.3
Changed lines of the file:
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@@
 		(lib_id "Device:R_Potentiometer_Small")
 		(at 173.99 67.31 0)
+		(mirror x)
 		(unit 1)
 		(exclude_from_sim no)
@@
 		(on_board yes)
 		(dnp no)
-		(fields_autoplaced yes)
 		(property "Reference" "R5"
-			(at 171.45 66.0399 0)
+			(at 171.45 68.5801 0)
 			(effects
 				(font
@@
 		)
 		(property "Value" "R5"
-			(at 171.45 68.5799 0)
+			(at 171.45 66.0401 0)
 			(effects
 				(font

Commit message: change potentiometer legs R5 and R33 again
Connections:
- net at U1.13 (PC2): now also R5.1; no longer R5.3
- net at R5.2, R6.1, U1.9 (VCOin): now also R5.3; no longer R5.1
Changed lines of the file:
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@@
 		(lib_id "Device:R_Potentiometer_Small")
 		(at 173.99 67.31 0)
-		(mirror x)
 		(unit 1)
 		(exclude_from_sim no)
@@
 		(dnp no)
 		(property "Reference" "R5"
-			(at 171.45 68.5801 0)
+			(at 171.45 66.0399 0)
 			(effects
 				(font
@@
 		)
 		(property "Value" "R5"
-			(at 171.45 66.0401 0)
+			(at 171.45 68.5799 0)
 			(effects
 				(font

Commit message: add Inhibit 4046
Parts:
- added J27: Inh, Connector_PinHeader_2.54mm:PinHeader_1x01_P2.54mm_Vertical, symbol Connector_Generic:Conn_01x01
Connections:
- net at R3.1, U1.5 (Inh): now also J27.1 (Pin_1)
Changed lines of the file:
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@@
+		(color 0 0 0 0)
+	)
+	(junction
+		(at 139.7 82.55)
+		(diameter 0)
 		(color 0 0 0 0)
 	)
@@
 					(unit 1)
 				)
+			)
+		)
+	)
+	(symbol
+		(lib_id "Connector_Generic:Conn_01x01")
+		(at 134.62 82.55 180)
+		(unit 1)
+		(exclude_from_sim no)
+		(in_bom yes)
+		(on_board yes)
+		(dnp no)
+		(property "Reference" "J27"
+			(at 134.62 76.962 0)
+			(effects
+				(font
+					(size 1.27 1.27)
+				)
+			)
+		)
+		(property "Value" "Inh"
+			(at 134.62 78.74 0)
+			(effects
+				(font
+					(size 1.27 1.27)
+				)
+			)
+		)
+		(property "Footprint" "Connector_PinHeader_2.54mm:PinHeader_1x01_P2.54mm_Vertical"
+			(at 134.62 82.55 0)
+			(effects
+				(font
+					(size 1.27 1.27)
+				)
+				(hide yes)
+			)
+		)
+		(property "Datasheet" "~"
+			(at 134.62 82.55 0)
+			(effects
+				(font
+					(size 1.27 1.27)
+				)
+				(hide yes)
+			)
+		)
+		(property "Description" "Generic connector, single row, 01x01, script generated (kicad-library-utils/schlib/autogen/connector/)"
+			(at 134.62 82.55 0)
+			(effects
+				(font
+					(size 1.27 1.27)
+				)
+				(hide yes)
+			)
+		)
+		(pin "1"
+		)
+		(instances
+			(project ""
+				(path "/01c1f2c1-4d06-4880-847a-9ab55552e3fd/79441be6-e853-4219-9c9d-5fa446c925d2"
+					(reference "J27")
+					(unit 1)
+				)
+				(path "/01c1f2c1-4d06-4880-847a-9ab55552e3fd/ec892350-7ee5-4574-b787-aa0418288502"
+					(reference "J28")
+					(unit 1)
+				)

Commit message: v2 initial commit
Parts:
- removed J27: Inh, Connector_PinHeader_2.54mm:PinHeader_1x01_P2.54mm_Vertical, symbol Connector_Generic:Conn_01x01
- added RV1: 2K, Potentiometer_THT:Potentiometer_Bourns_3296W_Vertical, symbol Device:R_Potentiometer_Trim
- added SW2: PLL Type, Button_Switch_THT:SW_E-Switch_EG1271_SPDT, symbol Switch:SW_SPDT
- renumbered C2 to C1, C1 to C2, R3 to R5, R5 to R6, R6 to R8, U1 to U2
Connections:
- net GND: now also RV1.3
- net SigIn: now also RV1.1, RV1.2
- net at R6.1: now also SW2.2 (B); no longer U2.13 (PC2)
- net at U2.2 (PC1): now also SW2.1 (A)
- net Inh: now reaches R5.1, U2.5 (Inh)
- new net: SW2.3 (C), U2.13 (PC2)
Other:
- moved on the sheet: C3, R6, R8
