File: 4046.kicad_sch (KiCad schematic)
At the start: 12 parts, among them SW6 PLL Type, SW9 SW_DPDT_x2, U9 4046

Commit message: drop 4040 outputs, rerouting
Parts:
- C25: value 100nF -> 10nF
- C5: value 10nF -> 1nF
- RV2: footprint Potentiometer_THT:Potentiometer_Bourns_3296W_Vertical -> Potentiometer_THT:Potentiometer_Bourns_3296Z_Horizontal
Changed lines of the file:
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@@
 			)
 		)
-		(property "Value" "100nF"
+		(property "Value" "10nF"
 			(at 99.06 77.4699 0)
 			(show_name no)
@@
 			)
 		)
-		(property "Value" "10nF"
+		(property "Value" "1nF"
 			(at 99.06 69.8499 0)
 			(show_name no)
@@
 			)
 		)
-		(property "Footprint" "Potentiometer_THT:Potentiometer_Bourns_3296W_Vertical"
+		(property "Footprint" "Potentiometer_THT:Potentiometer_Bourns_3296Z_Horizontal"
 			(at 83.82 73.66 0)
 			(hide yes)
