File: kleingorium.sync-conflict-20260322-030902-J4E24AU.kicad_pcb (KiCad board)
At the start: 2 copper layers, 500.1 x 100 mm, 179 parts, among them J1 VCC, J10 4046 Comp, J11 Select, J12 Select, J13 Inh, J14 Inh, J15 4046 Comp In, J16 4046 Comp In, J17 4046 Out, J18 4046 Out, J19 4040 Input, J2 VCC, J20 4040 Input, J21 4053 S3, J22 4053 S3, J23 4053 C, J24 4053 C, J25 4053 C0 C1, J26 4053 C0 C1, J27 4040 Output, J28 4040 Output, J29 4017 Fdbk, J3 GND, J30 4017 Fdbk, J31 Output, J32 Output, J33 4017 Pins, J34 4017 Pins, J35 Osc Out, J36 Conn_02x12_Odd_Even, J37 Conn_02x12_Odd_Even, J38 Conn_02x12_Odd_Even, J39 Conn_02x12_Odd_Even, J4 GND, J40 Conn_01x08, J41 Conn_01x08, J42 Osc Out, J43 Conn_02x08_Odd_Even, J44 Conn_02x08_Odd_Even, J45 Conn_02x08_Odd_Even, J46 Conn_02x08_Odd_Even, J47 Conn_02x08_Odd_Even, J48 Select, J49 Select, J5 Input, J50 Conn_02x18_Odd_Even, J51 Conn_02x18_Odd_Even, J52 Conn_02x18_Odd_Even, J53 Conn_02x18_Odd_Even, J54 Conn_02x18_Odd_Even, J55 01x18 from bottom plate, J56 VCC, J57 VCC, J58 GND, J59 GND, J6 Input, J60 VCC, J61 VCC, J62 GND, J63 GND, J64 Conn_02x08_Odd_Even, J65 Conn_02x18_Odd_Even, J66 4017 Pins, J67 4017 Pins, J68 Conn_01x16, J69 Conn_02x18_Odd_Even, J7 4046 SigIn, J70 Conn_02x18_Odd_Even, J71 Conn_02x18_Odd_Even, J73 Conn_02x20_Odd_Even, J74 Conn_02x20_Odd_Even, J75 Conn_02x20_Odd_Even, J76 Conn_02x20_Odd_Even, J77 Conn_02x20_Odd_Even, J78 Conn_02x20_Odd_Even, J79 Conn_02x20_Odd_Even, J8 4046 Comp, J80 Conn_02x20_Odd_Even, J81 Conn_02x20_Odd_Even, J83 Output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

Commit message: full alignment
Parts:
- removed J87: AudioJack3, Connector_Audio:Jack_3.5mm_CUI_SJ1-3523N_Horizontal
- added J72: Conn_02x18_Odd_Even, Connector_PinSocket_2.54mm:PinSocket_2x18_P2.54mm_Vertical, F.Cu at (565.7, -101.9)
- added J82: Conn_02x20_Odd_Even, Connector_PinHeader_2.54mm:PinHeader_2x20_P2.54mm_Vertical, F.Cu at (736.9, -101.9)
- moved U13 564.6 mm to (748.0, -93.0)
- moved R41 549.4 mm to (739.5, -21.4), turned to 0 degrees
- moved R38 549.1 mm to (739.5, -33.5), turned to 0 degrees
- moved J68 545.1 mm to (744.1, -101.8)
- moved J85 541.9 mm to (737.0, -49.0), turned to 0 degrees
- moved J62 538.3 mm to (729.9, -26.1)
- moved C22 536.0 mm to (739.5, -17.8)
- moved J61 532.0 mm to (729.9, -30.6)
- moved J42 529.1 mm to (729.9, -49.0)
- moved J48 529.0 mm to (729.9, -44.4)
- moved R40 526.1 mm to (739.5, -25.4)
- moved R39 525.9 mm to (739.5, -29.5)
- moved C20 501.5 mm to (711.2, -14.9), turned to 90 degrees
- moved R34 495.7 mm to (695.5, -14.9), turned to 90 degrees
- moved R36 492.7 mm to (703.6, -14.9), turned to 90 degrees
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Connections:
- J56 pad 1: VDDA -> Net-(J56-Pin_1)
- J56 pad 2: VDDA -> Net-(J56-Pin_1)
- J57 pad 1: VDDA -> Net-(J56-Pin_1)
- J57 pad 2: VDDA -> Net-(J56-Pin_1)
- J58 pad 1: GNDA -> Net-(J58-Pin_1)
- J58 pad 2: GNDA -> Net-(J58-Pin_1)
- J59 pad 1: GNDA -> Net-(J58-Pin_1)
- J59 pad 2: GNDA -> Net-(J58-Pin_1)
- J60 pad 1: VDDF -> Net-(J60-Pin_1)
- J60 pad 2: VDDF -> Net-(J60-Pin_1)
- J61 pad 1: VDDF -> Net-(J60-Pin_1)
- J61 pad 2: VDDF -> Net-(J60-Pin_1)
- J62 pad 1: GND2 -> Net-(J62-Pin_1)
- J62 pad 2: GND2 -> Net-(J62-Pin_1)
- J63 pad 1: GND2 -> Net-(J62-Pin_1)
- J63 pad 2: GND2 -> Net-(J62-Pin_1)
- J73 pad 21: Net-(J67-Pin_19) -> Net-(J67-Pin_1)
- J73 pad 22: Net-(J67-Pin_19) -> Net-(J67-Pin_1)
- J73 pad 23: Net-(J67-Pin_17) -> Net-(J67-Pin_3)
- J73 pad 24: Net-(J67-Pin_17) -> Net-(J67-Pin_3)
- J73 pad 25: Net-(J67-Pin_15) -> Net-(J67-Pin_5)
- J73 pad 26: Net-(J67-Pin_15) -> Net-(J67-Pin_5)
- J73 pad 27: Net-(J67-Pin_13) -> Net-(J67-Pin_7)
- J73 pad 28: Net-(J67-Pin_13) -> Net-(J67-Pin_7)
- J73 pad 29: Net-(J67-Pin_11) -> Net-(J67-Pin_10)
- J73 pad 30: Net-(J67-Pin_11) -> Net-(J67-Pin_10)
- J73 pad 31: Net-(J67-Pin_10) -> Net-(J67-Pin_11)
- J73 pad 32: Net-(J67-Pin_10) -> Net-(J67-Pin_11)
- J73 pad 33: Net-(J67-Pin_7) -> Net-(J67-Pin_13)
- J73 pad 34: Net-(J67-Pin_7) -> Net-(J67-Pin_13)
- J73 pad 35: Net-(J67-Pin_5) -> Net-(J67-Pin_15)
- J73 pad 36: Net-(J67-Pin_5) -> Net-(J67-Pin_15)
- J73 pad 37: Net-(J67-Pin_3) -> Net-(J67-Pin_17)
- J73 pad 38: Net-(J67-Pin_3) -> Net-(J67-Pin_17)
- J73 pad 39: Net-(J67-Pin_1) -> Net-(J67-Pin_19)
- J73 pad 40: Net-(J73-Pin_40) -> Net-(J67-Pin_19)
- J74 pad 21: Net-(J67-Pin_19) -> Net-(J67-Pin_1)
- J74 pad 22: Net-(J67-Pin_19) -> Net-(J67-Pin_1)
- J74 pad 23: Net-(J67-Pin_17) -> Net-(J67-Pin_3)
- J74 pad 24: Net-(J67-Pin_17) -> Net-(J67-Pin_3)
- J74 pad 25: Net-(J67-Pin_15) -> Net-(J67-Pin_5)
- J74 pad 26: Net-(J67-Pin_15) -> Net-(J67-Pin_5)
- J74 pad 27: Net-(J67-Pin_13) -> Net-(J67-Pin_7)
- J74 pad 28: Net-(J67-Pin_13) -> Net-(J67-Pin_7)
- J74 pad 29: Net-(J67-Pin_11) -> Net-(J67-Pin_10)
- J74 pad 30: Net-(J67-Pin_11) -> Net-(J67-Pin_10)
- J74 pad 31: Net-(J67-Pin_10) -> Net-(J67-Pin_11)
- J74 pad 32: Net-(J67-Pin_10) -> Net-(J67-Pin_11)
- J74 pad 33: Net-(J67-Pin_7) -> Net-(J67-Pin_13)
- J74 pad 34: Net-(J67-Pin_7) -> Net-(J67-Pin_13)
- J74 pad 35: Net-(J67-Pin_5) -> Net-(J67-Pin_15)
- J74 pad 36: Net-(J67-Pin_5) -> Net-(J67-Pin_15)
- J74 pad 37: Net-(J67-Pin_3) -> Net-(J67-Pin_17)
- J74 pad 38: Net-(J67-Pin_3) -> Net-(J67-Pin_17)
- J74 pad 39: Net-(J73-Pin_40) -> Net-(J67-Pin_19)
- J74 pad 40: Net-(J73-Pin_40) -> Net-(J67-Pin_19)
- J75 pad 21: Net-(J67-Pin_19) -> Net-(J67-Pin_1)
- J75 pad 22: Net-(J67-Pin_19) -> Net-(J67-Pin_1)
- J75 pad 23: Net-(J67-Pin_17) -> Net-(J67-Pin_3)
- J75 pad 24: Net-(J67-Pin_17) -> Net-(J67-Pin_3)
- J75 pad 25: Net-(J67-Pin_15) -> Net-(J67-Pin_5)
- J75 pad 26: Net-(J67-Pin_15) -> Net-(J67-Pin_5)
- J75 pad 27: Net-(J67-Pin_13) -> Net-(J67-Pin_7)
- J75 pad 28: Net-(J67-Pin_13) -> Net-(J67-Pin_7)
- J75 pad 29: Net-(J67-Pin_11) -> Net-(J67-Pin_10)
- J75 pad 30: Net-(J67-Pin_11) -> Net-(J67-Pin_10)
- J75 pad 31: Net-(J67-Pin_10) -> Net-(J67-Pin_11)
- J75 pad 32: Net-(J67-Pin_10) -> Net-(J67-Pin_11)
- J75 pad 33: Net-(J67-Pin_7) -> Net-(J67-Pin_13)
- J75 pad 34: Net-(J67-Pin_7) -> Net-(J67-Pin_13)
- J75 pad 35: Net-(J67-Pin_5) -> Net-(J67-Pin_15)
- J75 pad 36: Net-(J67-Pin_5) -> Net-(J67-Pin_15)
- J75 pad 37: Net-(J67-Pin_3) -> Net-(J67-Pin_17)
- J75 pad 38: Net-(J67-Pin_3) -> Net-(J67-Pin_17)
- J75 pad 39: Net-(J73-Pin_40) -> Net-(J67-Pin_19)
- J75 pad 40: Net-(J73-Pin_40) -> Net-(J67-Pin_19)
- J76 pad 21: Net-(J67-Pin_19) -> Net-(J67-Pin_1)
- J76 pad 22: Net-(J67-Pin_19) -> Net-(J67-Pin_1)
- J76 pad 23: Net-(J67-Pin_17) -> Net-(J67-Pin_3)
- J76 pad 24: Net-(J67-Pin_17) -> Net-(J67-Pin_3)
- J76 pad 25: Net-(J67-Pin_15) -> Net-(J67-Pin_5)
- J76 pad 26: Net-(J67-Pin_15) -> Net-(J67-Pin_5)
- J76 pad 27: Net-(J67-Pin_13) -> Net-(J67-Pin_7)
- J76 pad 28: Net-(J67-Pin_13) -> Net-(J67-Pin_7)
- J76 pad 29: Net-(J67-Pin_11) -> Net-(J67-Pin_10)
- J76 pad 30: Net-(J67-Pin_11) -> Net-(J67-Pin_10)
- J76 pad 31: Net-(J67-Pin_10) -> Net-(J67-Pin_11)
- J76 pad 32: Net-(J67-Pin_10) -> Net-(J67-Pin_11)
- J76 pad 33: Net-(J67-Pin_7) -> Net-(J67-Pin_13)
- J76 pad 34: Net-(J67-Pin_7) -> Net-(J67-Pin_13)
- J76 pad 35: Net-(J67-Pin_5) -> Net-(J67-Pin_15)
- J76 pad 36: Net-(J67-Pin_5) -> Net-(J67-Pin_15)
- J76 pad 37: Net-(J67-Pin_3) -> Net-(J67-Pin_17)
- J76 pad 38: Net-(J67-Pin_3) -> Net-(J67-Pin_17)
- J76 pad 39: Net-(J73-Pin_40) -> Net-(J67-Pin_19)
- J76 pad 40: Net-(J73-Pin_40) -> Net-(J67-Pin_19)
- J77 pad 21: Net-(J67-Pin_19) -> Net-(J67-Pin_1)
- J77 pad 22: Net-(J67-Pin_19) -> Net-(J67-Pin_1)
- J77 pad 23: Net-(J67-Pin_17) -> Net-(J67-Pin_3)
- J77 pad 24: Net-(J67-Pin_17) -> Net-(J67-Pin_3)
- J77 pad 25: Net-(J67-Pin_15) -> Net-(J67-Pin_5)
- J77 pad 26: Net-(J67-Pin_15) -> Net-(J67-Pin_5)
- J77 pad 27: Net-(J67-Pin_13) -> Net-(J67-Pin_7)
- J77 pad 28: Net-(J67-Pin_13) -> Net-(J67-Pin_7)
- J77 pad 29: Net-(J67-Pin_11) -> Net-(J67-Pin_10)
- J77 pad 30: Net-(J67-Pin_11) -> Net-(J67-Pin_10)
- J77 pad 31: Net-(J67-Pin_10) -> Net-(J67-Pin_11)
- J77 pad 32: Net-(J67-Pin_10) -> Net-(J67-Pin_11)
- J77 pad 33: Net-(J67-Pin_7) -> Net-(J67-Pin_13)
- J77 pad 34: Net-(J67-Pin_7) -> Net-(J67-Pin_13)
- J77 pad 35: Net-(J67-Pin_5) -> Net-(J67-Pin_15)
- J77 pad 36: Net-(J67-Pin_5) -> Net-(J67-Pin_15)
- J77 pad 37: Net-(J67-Pin_3) -> Net-(J67-Pin_17)
- J77 pad 38: Net-(J67-Pin_3) -> Net-(J67-Pin_17)
- J77 pad 39: Net-(J73-Pin_40) -> Net-(J67-Pin_19)
- J77 pad 40: Net-(J73-Pin_40) -> Net-(J67-Pin_19)
- J78 pad 21: Net-(J67-Pin_19) -> Net-(J67-Pin_1)
- J78 pad 22: Net-(J67-Pin_19) -> Net-(J67-Pin_1)
- J78 pad 23: Net-(J67-Pin_17) -> Net-(J67-Pin_3)
- J78 pad 24: Net-(J67-Pin_17) -> Net-(J67-Pin_3)
- J78 pad 25: Net-(J67-Pin_15) -> Net-(J67-Pin_5)
- J78 pad 26: Net-(J67-Pin_15) -> Net-(J67-Pin_5)
- J78 pad 27: Net-(J67-Pin_13) -> Net-(J67-Pin_7)
- J78 pad 28: Net-(J67-Pin_13) -> Net-(J67-Pin_7)
- J78 pad 29: Net-(J67-Pin_11) -> Net-(J67-Pin_10)
- J78 pad 30: Net-(J67-Pin_11) -> Net-(J67-Pin_10)
- J78 pad 31: Net-(J67-Pin_10) -> Net-(J67-Pin_11)
- J78 pad 32: Net-(J67-Pin_10) -> Net-(J67-Pin_11)
- J78 pad 33: Net-(J67-Pin_7) -> Net-(J67-Pin_13)
- J78 pad 34: Net-(J67-Pin_7) -> Net-(J67-Pin_13)
- J78 pad 35: Net-(J67-Pin_5) -> Net-(J67-Pin_15)
- J78 pad 36: Net-(J67-Pin_5) -> Net-(J67-Pin_15)
- J78 pad 37: Net-(J67-Pin_3) -> Net-(J67-Pin_17)
- J78 pad 38: Net-(J67-Pin_3) -> Net-(J67-Pin_17)
- J78 pad 39: Net-(J73-Pin_40) -> Net-(J67-Pin_19)
- J78 pad 40: Net-(J73-Pin_40) -> Net-(J67-Pin_19)
- J79 pad 21: Net-(J67-Pin_19) -> Net-(J67-Pin_1)
- J79 pad 22: Net-(J67-Pin_19) -> Net-(J67-Pin_1)
- J79 pad 23: Net-(J67-Pin_17) -> Net-(J67-Pin_3)
- J79 pad 24: Net-(J67-Pin_17) -> Net-(J67-Pin_3)
- J79 pad 25: Net-(J67-Pin_15) -> Net-(J67-Pin_5)
- J79 pad 26: Net-(J67-Pin_15) -> Net-(J67-Pin_5)
- J79 pad 27: Net-(J67-Pin_13) -> Net-(J67-Pin_7)
- J79 pad 28: Net-(J67-Pin_13) -> Net-(J67-Pin_7)
- J79 pad 29: Net-(J67-Pin_11) -> Net-(J67-Pin_10)
- J79 pad 30: Net-(J67-Pin_11) -> Net-(J67-Pin_10)
- J79 pad 31: Net-(J67-Pin_10) -> Net-(J67-Pin_11)
- J79 pad 32: Net-(J67-Pin_10) -> Net-(J67-Pin_11)
- J79 pad 33: Net-(J67-Pin_7) -> Net-(J67-Pin_13)
- J79 pad 34: Net-(J67-Pin_7) -> Net-(J67-Pin_13)
- J79 pad 35: Net-(J67-Pin_5) -> Net-(J67-Pin_15)
- J79 pad 36: Net-(J67-Pin_5) -> Net-(J67-Pin_15)
- J79 pad 37: Net-(J67-Pin_3) -> Net-(J67-Pin_17)
- J79 pad 38: Net-(J67-Pin_3) -> Net-(J67-Pin_17)
- J79 pad 39: Net-(J73-Pin_40) -> Net-(J67-Pin_19)
- J79 pad 40: Net-(J73-Pin_40) -> Net-(J67-Pin_19)
- J80 pad 21: Net-(J67-Pin_19) -> Net-(J67-Pin_1)
- J80 pad 22: Net-(J67-Pin_19) -> Net-(J67-Pin_1)
- J80 pad 23: Net-(J67-Pin_17) -> Net-(J67-Pin_3)
- J80 pad 24: Net-(J67-Pin_17) -> Net-(J67-Pin_3)
- J80 pad 25: Net-(J67-Pin_15) -> Net-(J67-Pin_5)
- J80 pad 26: Net-(J67-Pin_15) -> Net-(J67-Pin_5)
- J80 pad 27: Net-(J67-Pin_13) -> Net-(J67-Pin_7)
- J80 pad 28: Net-(J67-Pin_13) -> Net-(J67-Pin_7)
- J80 pad 29: Net-(J67-Pin_11) -> Net-(J67-Pin_10)
- J80 pad 30: Net-(J67-Pin_11) -> Net-(J67-Pin_10)
- J80 pad 31: Net-(J67-Pin_10) -> Net-(J67-Pin_11)
- J80 pad 32: Net-(J67-Pin_10) -> Net-(J67-Pin_11)
- J80 pad 33: Net-(J67-Pin_7) -> Net-(J67-Pin_13)
- J80 pad 34: Net-(J67-Pin_7) -> Net-(J67-Pin_13)
- J80 pad 35: Net-(J67-Pin_5) -> Net-(J67-Pin_15)
- J80 pad 36: Net-(J67-Pin_5) -> Net-(J67-Pin_15)
- J80 pad 37: Net-(J67-Pin_3) -> Net-(J67-Pin_17)
- J80 pad 38: Net-(J67-Pin_3) -> Net-(J67-Pin_17)
- J80 pad 39: Net-(J73-Pin_40) -> Net-(J67-Pin_19)
- J80 pad 40: Net-(J73-Pin_40) -> Net-(J67-Pin_19)
- J81 pad 21: Net-(J67-Pin_19) -> Net-(J67-Pin_1)
- J81 pad 22: Net-(J67-Pin_19) -> Net-(J67-Pin_1)
- J81 pad 23: Net-(J67-Pin_17) -> Net-(J67-Pin_3)
- J81 pad 24: Net-(J67-Pin_17) -> Net-(J67-Pin_3)
- J81 pad 25: Net-(J67-Pin_15) -> Net-(J67-Pin_5)
- J81 pad 26: Net-(J67-Pin_15) -> Net-(J67-Pin_5)
- J81 pad 27: Net-(J67-Pin_13) -> Net-(J67-Pin_7)
- J81 pad 28: Net-(J67-Pin_13) -> Net-(J67-Pin_7)
- J81 pad 29: Net-(J67-Pin_11) -> Net-(J67-Pin_10)
- J81 pad 30: Net-(J67-Pin_11) -> Net-(J67-Pin_10)
- J81 pad 31: Net-(J67-Pin_10) -> Net-(J67-Pin_11)
- J81 pad 32: Net-(J67-Pin_10) -> Net-(J67-Pin_11)
- J81 pad 33: Net-(J67-Pin_7) -> Net-(J67-Pin_13)
- J81 pad 34: Net-(J67-Pin_7) -> Net-(J67-Pin_13)
- J81 pad 35: Net-(J67-Pin_5) -> Net-(J67-Pin_15)
- J81 pad 36: Net-(J67-Pin_5) -> Net-(J67-Pin_15)
- J81 pad 37: Net-(J67-Pin_3) -> Net-(J67-Pin_17)
- J81 pad 38: Net-(J67-Pin_3) -> Net-(J67-Pin_17)
- J81 pad 39: Net-(J73-Pin_40) -> Net-(J67-Pin_19)
- J81 pad 40: Net-(J73-Pin_40) -> Net-(J67-Pin_19)
Routing:
- net /Multiplier-Divider/4520/Q1B: track 67.0 -> 5.88 mm
- net /Multiplier-Divider/4520/Q4A: track 57.8 -> 6.28 mm
- net /Multiplier-Divider/4520/Q4B: track 53.5 -> 5.88 mm
- net /Multiplier-Divider/4520/Q3A: track 53.7 -> 6.28 mm
- net /Multiplier-Divider/4520/Q3B: track 50.7 -> 5.88 mm
- net /Multiplier-Divider/4520/Q2A: track 50.1 -> 6.28 mm
- net /Multiplier-Divider/4520/Q1A: track 49.0 -> 6.28 mm
- net /Multiplier-Divider/4520/Q2B: track 46.7 -> 5.88 mm
- net Net-(U4A-Reset): track 14.4 -> 0.00 mm
- net /Multiplier-Divider/4520/CKA: track 22.3 -> 23.2 mm
- removed copper zone on B.Cu, net GND2
- removed copper zone on B.Cu, net GNDA
- removed copper zone on F.Cu, net VDDA
- removed copper zone on F.Cu, net VDDF
Other:
- board size 500.1 x 100 mm -> 722.5 x 373.2 mm
- copper layers 2 -> 4
- board text removed: "Bottom Plate"
- board text removed: "Top Plate"
- board text removed: "∞"
- board text removed: "𝅘𝅥𝅲 𝅘𝅥𝅱 𝅘𝅥𝅰 𝅘𝅥𝅯 𝅘𝅥𝅮 𝅘𝅥 𝅗𝅥 𝅝 𝅜 𝆷𝆶"
