File: 4017.kicad_sch (KiCad schematic)
At the start: 4 parts, among them U2 4017

Commit message: v2 initial commit
Parts:
- renumbered R10 to R1, R9 to R2, R8 to R3, U2 to U1
Changed lines of the file:
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@@
 		(dnp no)
 		(fields_autoplaced yes)
-		(property "Reference" "#PWR020"
+		(property "Reference" "#PWR03"
 			(at 134.62 119.38 0)
 			(effects
@@
 		(instances
 			(project "kleingorium"
-				(path "/01c1f2c1-4d06-4880-847a-9ab55552e3fd/2480befe-b8c4-416e-bc2e-ed39f97a6377"
-					(reference "#PWR020")
-					(unit 1)
-				)
-				(path "/01c1f2c1-4d06-4880-847a-9ab55552e3fd/b5613d46-8007-4aff-a7fe-9be23c91de99"
-					(reference "#PWR061")
+				(path "/01c1f2c1-4d06-4880-847a-9ab55552e3fd/ad1f1d92-237d-4bc3-883c-2ce266dd223f/69307ab1-0d8e-4901-8649-3291da88283b"
+					(reference "#PWR03")
 					(unit 1)
 				)
@@
 		(dnp no)
 		(fields_autoplaced yes)
-		(property "Reference" "R9"
+		(property "Reference" "R2"
 			(at 123.19 97.7899 0)
 			(effects
@@
 		(instances
 			(project "kleingorium"
-				(path "/01c1f2c1-4d06-4880-847a-9ab55552e3fd/2480befe-b8c4-416e-bc2e-ed39f97a6377"
-					(reference "R9")
-					(unit 1)
-				)
-				(path "/01c1f2c1-4d06-4880-847a-9ab55552e3fd/b5613d46-8007-4aff-a7fe-9be23c91de99"
-					(reference "R28")
+				(path "/01c1f2c1-4d06-4880-847a-9ab55552e3fd/ad1f1d92-237d-4bc3-883c-2ce266dd223f/69307ab1-0d8e-4901-8649-3291da88283b"
+					(reference "R2")
 					(unit 1)
 				)
@@
 		(dnp no)
 		(fields_autoplaced yes)
-		(property "Reference" "#PWR0102"
+		(property "Reference" "#PWR04"
 			(at 148.59 60.96 0)
 			(effects
@@
 		(instances
 			(project "kleingorium"
-				(path "/01c1f2c1-4d06-4880-847a-9ab55552e3fd/2480befe-b8c4-416e-bc2e-ed39f97a6377"
-					(reference "#PWR0102")
-					(unit 1)
-				)
-				(path "/01c1f2c1-4d06-4880-847a-9ab55552e3fd/b5613d46-8007-4aff-a7fe-9be23c91de99"
-					(reference "#PWR065")
+				(path "/01c1f2c1-4d06-4880-847a-9ab55552e3fd/ad1f1d92-237d-4bc3-883c-2ce266dd223f/69307ab1-0d8e-4901-8649-3291da88283b"
+					(reference "#PWR04")
 					(unit 1)
 				)
@@
 		(dnp no)
 		(fields_autoplaced yes)
-		(property "Reference" "#PWR027"
+		(property "Reference" "#PWR05"
 			(at 148.59 119.38 0)
 			(effects
@@
 		(instances
 			(project "kleingorium"
-				(path "/01c1f2c1-4d06-4880-847a-9ab55552e3fd/2480befe-b8c4-416e-bc2e-ed39f97a6377"
-					(reference "#PWR027")
-					(unit 1)
-				)
-				(path "/01c1f2c1-4d06-4880-847a-9ab55552e3fd/b5613d46-8007-4aff-a7fe-9be23c91de99"
-					(reference "#PWR066")
+				(path "/01c1f2c1-4d06-4880-847a-9ab55552e3fd/ad1f1d92-237d-4bc3-883c-2ce266dd223f/69307ab1-0d8e-4901-8649-3291da88283b"
+					(reference "#PWR05")
 					(unit 1)
 				)
@@
 		(dnp no)
 		(fields_autoplaced yes)
-		(property "Reference" "U2"
+		(property "Reference" "U1"
 			(at 150.7333 57.15 0)
 			(effects
@@
 		(instances
 			(project "kleingorium"
-				(path "/01c1f2c1-4d06-4880-847a-9ab55552e3fd/2480befe-b8c4-416e-bc2e-ed39f97a6377"
-					(reference "U2")
-					(unit 1)
-				)
-				(path "/01c1f2c1-4d06-4880-847a-9ab55552e3fd/b5613d46-8007-4aff-a7fe-9be23c91de99"
-					(reference "U14")
+				(path "/01c1f2c1-4d06-4880-847a-9ab55552e3fd/ad1f1d92-237d-4bc3-883c-2ce266dd223f/69307ab1-0d8e-4901-8649-3291da88283b"
+					(reference "U1")
 					(unit 1)
 				)
@@
 		(dnp no)
 		(fields_autoplaced yes)
-		(property "Reference" "R8"
+		(property "Reference" "R3"
 			(at 137.16 102.8699 0)
 			(effects
@@
 		(instances
 			(project "kleingorium"
-				(path "/01c1f2c1-4d06-4880-847a-9ab55552e3fd/2480befe-b8c4-416e-bc2e-ed39f97a6377"
-					(reference "R8")
-					(unit 1)
-				)
-				(path "/01c1f2c1-4d06-4880-847a-9ab55552e3fd/b5613d46-8007-4aff-a7fe-9be23c91de99"
-					(reference "R31")
+				(path "/01c1f2c1-4d06-4880-847a-9ab55552e3fd/ad1f1d92-237d-4bc3-883c-2ce266dd223f/69307ab1-0d8e-4901-8649-3291da88283b"
+					(reference "R3")
 					(unit 1)
 				)
@@
 		(dnp no)
 		(fields_autoplaced yes)
-		(property "Reference" "R10"
+		(property "Reference" "R1"
 			(at 102.87 95.2499 0)
 			(effects
@@
 		(instances
 			(project "kleingorium"
-				(path "/01c1f2c1-4d06-4880-847a-9ab55552e3fd/2480befe-b8c4-416e-bc2e-ed39f97a6377"
-					(reference "R10")
-					(unit 1)
-				)
-				(path "/01c1f2c1-4d06-4880-847a-9ab55552e3fd/b5613d46-8007-4aff-a7fe-9be23c91de99"
-					(reference "R25")
+				(path "/01c1f2c1-4d06-4880-847a-9ab55552e3fd/ad1f1d92-237d-4bc3-883c-2ce266dd223f/69307ab1-0d8e-4901-8649-3291da88283b"
+					(reference "R1")
 					(unit 1)
 				)
@@
 		(dnp no)
 		(fields_autoplaced yes)
-		(property "Reference" "#PWR022"
+		(property "Reference" "#PWR01"
 			(at 100.33 111.76 0)
 			(effects
@@
 		(instances
 			(project "kleingorium"
-				(path "/01c1f2c1-4d06-4880-847a-9ab55552e3fd/2480befe-b8c4-416e-bc2e-ed39f97a6377"
-					(reference "#PWR022")
-					(unit 1)
-				)
-				(path "/01c1f2c1-4d06-4880-847a-9ab55552e3fd/b5613d46-8007-4aff-a7fe-9be23c91de99"
-					(reference "#PWR046")
+				(path "/01c1f2c1-4d06-4880-847a-9ab55552e3fd/ad1f1d92-237d-4bc3-883c-2ce266dd223f/69307ab1-0d8e-4901-8649-3291da88283b"
+					(reference "#PWR01")
 					(unit 1)
 				)
@@
 		(dnp no)
 		(fields_autoplaced yes)
-		(property "Reference" "#PWR021"
+		(property "Reference" "#PWR02"
 			(at 120.65 114.3 0)
 			(effects
@@
 		(instances
 			(project "kleingorium"
-				(path "/01c1f2c1-4d06-4880-847a-9ab55552e3fd/2480befe-b8c4-416e-bc2e-ed39f97a6377"
-					(reference "#PWR021")
-					(unit 1)
-				)
-				(path "/01c1f2c1-4d06-4880-847a-9ab55552e3fd/b5613d46-8007-4aff-a7fe-9be23c91de99"
-					(reference "#PWR049")
-					(unit 1)
-				)
+				(path "/01c1f2c1-4d06-4880-847a-9ab55552e3fd/ad1f1d92-237d-4bc3-883c-2ce266dd223f/69307ab1-0d8e-4901-8649-3291da88283b"
+					(reference "#PWR02")
+					(unit 1)
+				)

Commit message: schematic finished
Parts:
- renumbered R1 to R3, R2 to R4, R3 to R5
Connections:
- net Q10: no longer names the net of U1.12 (Cout)
Changed lines of the file:
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@@
-	(wire
-		(pts
-			(xy 161.29 92.71) (xy 167.64 92.71)
-		)
-		(stroke
-			(width 0)
-			(type default)
-		)
-	)
 	(wire
 		(pts
@@
 		(shape input)
 		(at 167.64 77.47 0)
-		(effects
-			(font
-				(size 1.27 1.27)
-			)
-			(justify left)
-		)
-	)
-	(hierarchical_label "Q10"
-		(shape input)
-		(at 167.64 92.71 0)
 		(effects
 			(font
@@
 		(dnp no)
 		(fields_autoplaced yes)
-		(property "Reference" "#PWR03"
+		(property "Reference" "#PWR07"
 			(at 134.62 119.38 0)
 			(effects
@@
 		(instances
 			(project "kleingorium"
+				(path "/01c1f2c1-4d06-4880-847a-9ab55552e3fd/ad1f1d92-237d-4bc3-883c-2ce266dd223f/4ed119e9-593d-4415-8ac1-9a66b84ab373"
+					(reference "#PWR039")
+					(unit 1)
+				)
 				(path "/01c1f2c1-4d06-4880-847a-9ab55552e3fd/ad1f1d92-237d-4bc3-883c-2ce266dd223f/69307ab1-0d8e-4901-8649-3291da88283b"
-					(reference "#PWR03")
+					(reference "#PWR07")
 					(unit 1)
 				)
@@
 		(dnp no)
 		(fields_autoplaced yes)
-		(property "Reference" "R2"
+		(property "Reference" "R4"
 			(at 123.19 97.7899 0)
 			(effects
@@
 		(instances
 			(project "kleingorium"
+				(path "/01c1f2c1-4d06-4880-847a-9ab55552e3fd/ad1f1d92-237d-4bc3-883c-2ce266dd223f/4ed119e9-593d-4415-8ac1-9a66b84ab373"
+					(reference "R23")
+					(unit 1)
+				)
 				(path "/01c1f2c1-4d06-4880-847a-9ab55552e3fd/ad1f1d92-237d-4bc3-883c-2ce266dd223f/69307ab1-0d8e-4901-8649-3291da88283b"
-					(reference "R2")
+					(reference "R4")
 					(unit 1)
 				)
@@
 		(dnp no)
 		(fields_autoplaced yes)
-		(property "Reference" "#PWR04"
+		(property "Reference" "#PWR012"
 			(at 148.59 60.96 0)
 			(effects
@@
 		(instances
 			(project "kleingorium"
+				(path "/01c1f2c1-4d06-4880-847a-9ab55552e3fd/ad1f1d92-237d-4bc3-883c-2ce266dd223f/4ed119e9-593d-4415-8ac1-9a66b84ab373"
+					(reference "#PWR040")
+					(unit 1)
+				)
 				(path "/01c1f2c1-4d06-4880-847a-9ab55552e3fd/ad1f1d92-237d-4bc3-883c-2ce266dd223f/69307ab1-0d8e-4901-8649-3291da88283b"
-					(reference "#PWR04")
+					(reference "#PWR012")
 					(unit 1)
 				)
@@
 		(dnp no)
 		(fields_autoplaced yes)
-		(property "Reference" "#PWR05"
+		(property "Reference" "#PWR013"
 			(at 148.59 119.38 0)
 			(effects
@@
 		(instances
 			(project "kleingorium"
+				(path "/01c1f2c1-4d06-4880-847a-9ab55552e3fd/ad1f1d92-237d-4bc3-883c-2ce266dd223f/4ed119e9-593d-4415-8ac1-9a66b84ab373"
+					(reference "#PWR041")
+					(unit 1)
+				)
 				(path "/01c1f2c1-4d06-4880-847a-9ab55552e3fd/ad1f1d92-237d-4bc3-883c-2ce266dd223f/69307ab1-0d8e-4901-8649-3291da88283b"
-					(reference "#PWR05")
+					(reference "#PWR013")
 					(unit 1)
 				)
@@
 		(instances
 			(project "kleingorium"
+				(path "/01c1f2c1-4d06-4880-847a-9ab55552e3fd/ad1f1d92-237d-4bc3-883c-2ce266dd223f/4ed119e9-593d-4415-8ac1-9a66b84ab373"
+					(reference "U6")
+					(unit 1)
+				)
 				(path "/01c1f2c1-4d06-4880-847a-9ab55552e3fd/ad1f1d92-237d-4bc3-883c-2ce266dd223f/69307ab1-0d8e-4901-8649-3291da88283b"
 					(reference "U1")
@@
 		(dnp no)
 		(fields_autoplaced yes)
-		(property "Reference" "R3"
+		(property "Reference" "R5"
 			(at 137.16 102.8699 0)
 			(effects
@@
 		(instances
 			(project "kleingorium"
+				(path "/01c1f2c1-4d06-4880-847a-9ab55552e3fd/ad1f1d92-237d-4bc3-883c-2ce266dd223f/4ed119e9-593d-4415-8ac1-9a66b84ab373"
+					(reference "R24")
+					(unit 1)
+				)
 				(path "/01c1f2c1-4d06-4880-847a-9ab55552e3fd/ad1f1d92-237d-4bc3-883c-2ce266dd223f/69307ab1-0d8e-4901-8649-3291da88283b"
-					(reference "R3")
+					(reference "R5")
 					(unit 1)
 				)
@@
 		(dnp no)
 		(fields_autoplaced yes)
-		(property "Reference" "R1"
+		(property "Reference" "R3"
 			(at 102.87 95.2499 0)
 			(effects
@@
 		(instances
 			(project "kleingorium"
+				(path "/01c1f2c1-4d06-4880-847a-9ab55552e3fd/ad1f1d92-237d-4bc3-883c-2ce266dd223f/4ed119e9-593d-4415-8ac1-9a66b84ab373"
+					(reference "R22")
+					(unit 1)
+				)
 				(path "/01c1f2c1-4d06-4880-847a-9ab55552e3fd/ad1f1d92-237d-4bc3-883c-2ce266dd223f/69307ab1-0d8e-4901-8649-3291da88283b"
-					(reference "R1")
+					(reference "R3")
 					(unit 1)
 				)
@@
 		(dnp no)
 		(fields_autoplaced yes)
-		(property "Reference" "#PWR01"
+		(property "Reference" "#PWR05"
 			(at 100.33 111.76 0)
 			(effects
@@
 		(instances
 			(project "kleingorium"
+				(path "/01c1f2c1-4d06-4880-847a-9ab55552e3fd/ad1f1d92-237d-4bc3-883c-2ce266dd223f/4ed119e9-593d-4415-8ac1-9a66b84ab373"
+					(reference "#PWR037")
+					(unit 1)
+				)
 				(path "/01c1f2c1-4d06-4880-847a-9ab55552e3fd/ad1f1d92-237d-4bc3-883c-2ce266dd223f/69307ab1-0d8e-4901-8649-3291da88283b"
-					(reference "#PWR01")
+					(reference "#PWR05")
 					(unit 1)
 				)
@@
 		(dnp no)
 		(fields_autoplaced yes)
-		(property "Reference" "#PWR02"
+		(property "Reference" "#PWR06"
 			(at 120.65 114.3 0)
 			(effects
@@
 		(instances
 			(project "kleingorium"
+				(path "/01c1f2c1-4d06-4880-847a-9ab55552e3fd/ad1f1d92-237d-4bc3-883c-2ce266dd223f/4ed119e9-593d-4415-8ac1-9a66b84ab373"
+					(reference "#PWR038")
+					(unit 1)
+				)
 				(path "/01c1f2c1-4d06-4880-847a-9ab55552e3fd/ad1f1d92-237d-4bc3-883c-2ce266dd223f/69307ab1-0d8e-4901-8649-3291da88283b"
-					(reference "#PWR02")
-					(unit 1)
-				)
+					(reference "#PWR06")
+					(unit 1)
+				)

Commit message: wip symmetric layout
Parts:
- renumbered R3 to R24, R4 to R25, R5 to R26, U1 to U8
Changed lines of the file:
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@@
 		(dnp no)
 		(fields_autoplaced yes)
-		(property "Reference" "#PWR07"
+		(property "Reference" "#PWR044"
 			(at 134.62 119.38 0)
 			(effects
@@
 		(instances
 			(project "kleingorium"
-				(path "/01c1f2c1-4d06-4880-847a-9ab55552e3fd/ad1f1d92-237d-4bc3-883c-2ce266dd223f/4ed119e9-593d-4415-8ac1-9a66b84ab373"
-					(reference "#PWR039")
-					(unit 1)
-				)
-				(path "/01c1f2c1-4d06-4880-847a-9ab55552e3fd/ad1f1d92-237d-4bc3-883c-2ce266dd223f/69307ab1-0d8e-4901-8649-3291da88283b"
-					(reference "#PWR07")
+				(path "/01c1f2c1-4d06-4880-847a-9ab55552e3fd/ad1f1d92-237d-4bc3-883c-2ce266dd223f/4b203833-f0af-4e88-a9fb-191df5175df3/09e0e8a4-54b2-4381-b75b-b44baf0b4473"
+					(reference "#PWR05")
+					(unit 1)
+				)
+				(path "/01c1f2c1-4d06-4880-847a-9ab55552e3fd/ad1f1d92-237d-4bc3-883c-2ce266dd223f/e00ebc01-440e-4477-8d51-aed2c51c95ea/09e0e8a4-54b2-4381-b75b-b44baf0b4473"
+					(reference "#PWR044")
 					(unit 1)
 				)
@@
 		(dnp no)
 		(fields_autoplaced yes)
-		(property "Reference" "R4"
+		(property "Reference" "R25"
 			(at 123.19 97.7899 0)
 			(effects
@@
 		(instances
 			(project "kleingorium"
-				(path "/01c1f2c1-4d06-4880-847a-9ab55552e3fd/ad1f1d92-237d-4bc3-883c-2ce266dd223f/4ed119e9-593d-4415-8ac1-9a66b84ab373"
-					(reference "R23")
-					(unit 1)
-				)
-				(path "/01c1f2c1-4d06-4880-847a-9ab55552e3fd/ad1f1d92-237d-4bc3-883c-2ce266dd223f/69307ab1-0d8e-4901-8649-3291da88283b"
-					(reference "R4")
+				(path "/01c1f2c1-4d06-4880-847a-9ab55552e3fd/ad1f1d92-237d-4bc3-883c-2ce266dd223f/4b203833-f0af-4e88-a9fb-191df5175df3/09e0e8a4-54b2-4381-b75b-b44baf0b4473"
+					(reference "R3")
+					(unit 1)
+				)
+				(path "/01c1f2c1-4d06-4880-847a-9ab55552e3fd/ad1f1d92-237d-4bc3-883c-2ce266dd223f/e00ebc01-440e-4477-8d51-aed2c51c95ea/09e0e8a4-54b2-4381-b75b-b44baf0b4473"
+					(reference "R25")
 					(unit 1)
 				)
@@
 		(dnp no)
 		(fields_autoplaced yes)
-		(property "Reference" "#PWR012"
+		(property "Reference" "#PWR045"
 			(at 148.59 60.96 0)
 			(effects
@@
 		(instances
 			(project "kleingorium"
-				(path "/01c1f2c1-4d06-4880-847a-9ab55552e3fd/ad1f1d92-237d-4bc3-883c-2ce266dd223f/4ed119e9-593d-4415-8ac1-9a66b84ab373"
-					(reference "#PWR040")
-					(unit 1)
-				)
-				(path "/01c1f2c1-4d06-4880-847a-9ab55552e3fd/ad1f1d92-237d-4bc3-883c-2ce266dd223f/69307ab1-0d8e-4901-8649-3291da88283b"
-					(reference "#PWR012")
+				(path "/01c1f2c1-4d06-4880-847a-9ab55552e3fd/ad1f1d92-237d-4bc3-883c-2ce266dd223f/4b203833-f0af-4e88-a9fb-191df5175df3/09e0e8a4-54b2-4381-b75b-b44baf0b4473"
+					(reference "#PWR06")
+					(unit 1)
+				)
+				(path "/01c1f2c1-4d06-4880-847a-9ab55552e3fd/ad1f1d92-237d-4bc3-883c-2ce266dd223f/e00ebc01-440e-4477-8d51-aed2c51c95ea/09e0e8a4-54b2-4381-b75b-b44baf0b4473"
+					(reference "#PWR045")
 					(unit 1)
 				)
@@
 		(dnp no)
 		(fields_autoplaced yes)
-		(property "Reference" "#PWR013"
+		(property "Reference" "#PWR046"
 			(at 148.59 119.38 0)
 			(effects
@@
 		(instances
 			(project "kleingorium"
-				(path "/01c1f2c1-4d06-4880-847a-9ab55552e3fd/ad1f1d92-237d-4bc3-883c-2ce266dd223f/4ed119e9-593d-4415-8ac1-9a66b84ab373"
-					(reference "#PWR041")
-					(unit 1)
-				)
-				(path "/01c1f2c1-4d06-4880-847a-9ab55552e3fd/ad1f1d92-237d-4bc3-883c-2ce266dd223f/69307ab1-0d8e-4901-8649-3291da88283b"
-					(reference "#PWR013")
+				(path "/01c1f2c1-4d06-4880-847a-9ab55552e3fd/ad1f1d92-237d-4bc3-883c-2ce266dd223f/4b203833-f0af-4e88-a9fb-191df5175df3/09e0e8a4-54b2-4381-b75b-b44baf0b4473"
+					(reference "#PWR07")
+					(unit 1)
+				)
+				(path "/01c1f2c1-4d06-4880-847a-9ab55552e3fd/ad1f1d92-237d-4bc3-883c-2ce266dd223f/e00ebc01-440e-4477-8d51-aed2c51c95ea/09e0e8a4-54b2-4381-b75b-b44baf0b4473"
+					(reference "#PWR046")
 					(unit 1)
 				)
@@
 		(dnp no)
 		(fields_autoplaced yes)
-		(property "Reference" "U1"
+		(property "Reference" "U8"
 			(at 150.7333 57.15 0)
 			(effects
@@
 		(instances
 			(project "kleingorium"
-				(path "/01c1f2c1-4d06-4880-847a-9ab55552e3fd/ad1f1d92-237d-4bc3-883c-2ce266dd223f/4ed119e9-593d-4415-8ac1-9a66b84ab373"
-					(reference "U6")
-					(unit 1)
-				)
-				(path "/01c1f2c1-4d06-4880-847a-9ab55552e3fd/ad1f1d92-237d-4bc3-883c-2ce266dd223f/69307ab1-0d8e-4901-8649-3291da88283b"
+				(path "/01c1f2c1-4d06-4880-847a-9ab55552e3fd/ad1f1d92-237d-4bc3-883c-2ce266dd223f/4b203833-f0af-4e88-a9fb-191df5175df3/09e0e8a4-54b2-4381-b75b-b44baf0b4473"
 					(reference "U1")
+					(unit 1)
+				)
+				(path "/01c1f2c1-4d06-4880-847a-9ab55552e3fd/ad1f1d92-237d-4bc3-883c-2ce266dd223f/e00ebc01-440e-4477-8d51-aed2c51c95ea/09e0e8a4-54b2-4381-b75b-b44baf0b4473"
+					(reference "U8")
 					(unit 1)
 				)
@@
 		(dnp no)
 		(fields_autoplaced yes)
-		(property "Reference" "R5"
+		(property "Reference" "R26"
 			(at 137.16 102.8699 0)
 			(effects
@@
 		(instances
 			(project "kleingorium"
-				(path "/01c1f2c1-4d06-4880-847a-9ab55552e3fd/ad1f1d92-237d-4bc3-883c-2ce266dd223f/4ed119e9-593d-4415-8ac1-9a66b84ab373"
-					(reference "R24")
-					(unit 1)
-				)
-				(path "/01c1f2c1-4d06-4880-847a-9ab55552e3fd/ad1f1d92-237d-4bc3-883c-2ce266dd223f/69307ab1-0d8e-4901-8649-3291da88283b"
-					(reference "R5")
+				(path "/01c1f2c1-4d06-4880-847a-9ab55552e3fd/ad1f1d92-237d-4bc3-883c-2ce266dd223f/4b203833-f0af-4e88-a9fb-191df5175df3/09e0e8a4-54b2-4381-b75b-b44baf0b4473"
+					(reference "R4")
+					(unit 1)
+				)
+				(path "/01c1f2c1-4d06-4880-847a-9ab55552e3fd/ad1f1d92-237d-4bc3-883c-2ce266dd223f/e00ebc01-440e-4477-8d51-aed2c51c95ea/09e0e8a4-54b2-4381-b75b-b44baf0b4473"
+					(reference "R26")
 					(unit 1)
 				)
@@
 		(dnp no)
 		(fields_autoplaced yes)
-		(property "Reference" "R3"
+		(property "Reference" "R24"
 			(at 102.87 95.2499 0)
 			(effects
@@
 		(instances
 			(project "kleingorium"
-				(path "/01c1f2c1-4d06-4880-847a-9ab55552e3fd/ad1f1d92-237d-4bc3-883c-2ce266dd223f/4ed119e9-593d-4415-8ac1-9a66b84ab373"
-					(reference "R22")
-					(unit 1)
-				)
-				(path "/01c1f2c1-4d06-4880-847a-9ab55552e3fd/ad1f1d92-237d-4bc3-883c-2ce266dd223f/69307ab1-0d8e-4901-8649-3291da88283b"
-					(reference "R3")
+				(path "/01c1f2c1-4d06-4880-847a-9ab55552e3fd/ad1f1d92-237d-4bc3-883c-2ce266dd223f/4b203833-f0af-4e88-a9fb-191df5175df3/09e0e8a4-54b2-4381-b75b-b44baf0b4473"
+					(reference "R2")
+					(unit 1)
+				)
+				(path "/01c1f2c1-4d06-4880-847a-9ab55552e3fd/ad1f1d92-237d-4bc3-883c-2ce266dd223f/e00ebc01-440e-4477-8d51-aed2c51c95ea/09e0e8a4-54b2-4381-b75b-b44baf0b4473"
+					(reference "R24")
 					(unit 1)
 				)
@@
 		(dnp no)
 		(fields_autoplaced yes)
-		(property "Reference" "#PWR05"
+		(property "Reference" "#PWR042"
 			(at 100.33 111.76 0)
 			(effects
@@
 		(instances
 			(project "kleingorium"
-				(path "/01c1f2c1-4d06-4880-847a-9ab55552e3fd/ad1f1d92-237d-4bc3-883c-2ce266dd223f/4ed119e9-593d-4415-8ac1-9a66b84ab373"
-					(reference "#PWR037")
-					(unit 1)
-				)
-				(path "/01c1f2c1-4d06-4880-847a-9ab55552e3fd/ad1f1d92-237d-4bc3-883c-2ce266dd223f/69307ab1-0d8e-4901-8649-3291da88283b"
-					(reference "#PWR05")
+				(path "/01c1f2c1-4d06-4880-847a-9ab55552e3fd/ad1f1d92-237d-4bc3-883c-2ce266dd223f/4b203833-f0af-4e88-a9fb-191df5175df3/09e0e8a4-54b2-4381-b75b-b44baf0b4473"
+					(reference "#PWR03")
+					(unit 1)
+				)
+				(path "/01c1f2c1-4d06-4880-847a-9ab55552e3fd/ad1f1d92-237d-4bc3-883c-2ce266dd223f/e00ebc01-440e-4477-8d51-aed2c51c95ea/09e0e8a4-54b2-4381-b75b-b44baf0b4473"
+					(reference "#PWR042")
 					(unit 1)
 				)
@@
 		(dnp no)
 		(fields_autoplaced yes)
-		(property "Reference" "#PWR06"
+		(property "Reference" "#PWR043"
 			(at 120.65 114.3 0)
 			(effects
@@
 		(instances
 			(project "kleingorium"
-				(path "/01c1f2c1-4d06-4880-847a-9ab55552e3fd/ad1f1d92-237d-4bc3-883c-2ce266dd223f/4ed119e9-593d-4415-8ac1-9a66b84ab373"
-					(reference "#PWR038")
-					(unit 1)
-				)
-				(path "/01c1f2c1-4d06-4880-847a-9ab55552e3fd/ad1f1d92-237d-4bc3-883c-2ce266dd223f/69307ab1-0d8e-4901-8649-3291da88283b"
-					(reference "#PWR06")
-					(unit 1)
-				)
+				(path "/01c1f2c1-4d06-4880-847a-9ab55552e3fd/ad1f1d92-237d-4bc3-883c-2ce266dd223f/4b203833-f0af-4e88-a9fb-191df5175df3/09e0e8a4-54b2-4381-b75b-b44baf0b4473"
+					(reference "#PWR04")
+					(unit 1)
+				)
+				(path "/01c1f2c1-4d06-4880-847a-9ab55552e3fd/ad1f1d92-237d-4bc3-883c-2ce266dd223f/e00ebc01-440e-4477-8d51-aed2c51c95ea/09e0e8a4-54b2-4381-b75b-b44baf0b4473"
+					(reference "#PWR043")
+					(unit 1)
+				)
