File: 4040_2.kicad_sch (KiCad schematic)
At the start: 2 parts, among them U3 4040

Commit message: schematic finished
Parts:
- removed R12: 100K, Resistor_THT:R_Axial_DIN0207_L6.3mm_D2.5mm_P10.16mm_Horizontal, symbol Device:R_Small
- removed U3: 4040, Package_DIP:DIP-16_W7.62mm, symbol 4xxx:4040
- added C21: 100nF, Capacitor_THT:C_Disc_D3.0mm_W1.6mm_P2.50mm, symbol Device:C_Small
- added R33: 100K, Resistor_THT:R_Axial_DIN0207_L6.3mm_D2.5mm_P10.16mm_Horizontal, symbol Device:R_Small
- added U11: 4040, Package_DIP:DIP-16_W7.62mm, symbol 4xxx:4040
Connections:
- net Clock: now also U11.10 (CLK)
- net Q0: now also U11.9 (Q0)
- net Q1: now also U11.7 (Q1)
- net Q10: now also U11.15 (Q10)
- net Q11: now also U11.1 (Q11)
- net Q2: now also U11.6 (Q2)
- net Q3: now also U11.5 (Q3)
- net Q4: now also U11.3 (Q4)
- net Q5: now also U11.2 (Q5)
- net Q6: now also U11.4 (Q6)
- net Q7: now also U11.13 (Q7)
- net Q8: now also U11.12 (Q8)
- net Q9: now also U11.14 (Q9)
- net Reset: now also R33.1, U11.11 (Reset)
- new net GNDA: C21.2, R33.2, U11.8 (VSS)
- new net VDDA: C21.1, U11.16 (VDD)
