File: 4040_2.kicad_sch (KiCad schematic)
At the start: 3 parts, among them U11 4040

Commit message: start smd refactoring
Parts:
- C21: footprint Capacitor_THT:C_Disc_D3.0mm_W1.6mm_P2.50mm -> C_0805_2012Metric; KiLib_Generator (none) -> SMD_2terminal_chip_molded
- R33: footprint Resistor_THT:R_Axial_DIN0207_L6.3mm_D2.5mm_P10.16mm_Horizontal -> R_0805_2012Metric; KiLib_Generator (none) -> SMD_2terminal_chip_molded
- U11: footprint Package_DIP:DIP-16_W7.62mm -> SOIC-16_3.9x9.9mm_P1.27mm; KiLib_Generator (none) -> package/gullwing
Changed lines of the file:
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@@
 			)
 		)
-		(property "Footprint" "Capacitor_THT:C_Disc_D3.0mm_W1.6mm_P2.50mm"
+		(property "Footprint" "C_0805_2012Metric"
 			(at 151.13 46.99 0)
 			(hide yes)
@@
 			)
 		)
-		(property "Description" "Unpolarized capacitor, small symbol"
+		(property "Description" ""
+			(at 151.13 46.99 0)
+			(hide yes)
+			(show_name no)
+			(do_not_autoplace no)
+			(effects
+				(font
+					(size 1.27 1.27)
+				)
+			)
+		)
+		(property "KiLib_Generator" "SMD_2terminal_chip_molded"
 			(at 151.13 46.99 0)
 			(hide yes)
@@
 			)
 		)
-		(property "Footprint" "Package_DIP:DIP-16_W7.62mm"
+		(property "Footprint" "SOIC-16_3.9x9.9mm_P1.27mm"
 			(at 133.35 69.85 0)
 			(hide yes)
@@
 			)
 		)
-		(property "Datasheet" "http://www.intersil.com/content/dam/Intersil/documents/cd40/cd4020bms-24bms-40bms.pdf"
+		(property "Datasheet" ""
 			(at 133.35 69.85 0)
 			(hide yes)
@@
 			)
 		)
-		(property "Description" "Binary Counter 12 stages (Asynchronous)"
+		(property "Description" ""
+			(at 133.35 69.85 0)
+			(hide yes)
+			(show_name no)
+			(do_not_autoplace no)
+			(effects
+				(font
+					(size 1.27 1.27)
+				)
+			)
+		)
+		(property "KiLib_Generator" "package/gullwing"
 			(at 133.35 69.85 0)
 			(hide yes)
@@
 			)
 		)
-		(property "Footprint" "Resistor_THT:R_Axial_DIN0207_L6.3mm_D2.5mm_P10.16mm_Horizontal"
+		(property "Footprint" "R_0805_2012Metric"
 			(at 116.84 76.2 0)
 			(hide yes)
@@
 			)
 		)
-		(property "Description" "Resistor, small symbol"
+		(property "Description" ""
 			(at 116.84 76.2 0)
 			(hide yes)
+			(show_name no)
+			(do_not_autoplace no)
+			(effects
+				(font
+					(size 1.27 1.27)
+				)
+			)
+		)
+		(property "KiLib_Generator" "SMD_2terminal_chip_molded"
+			(at 116.84 76.2 0)
+			(hide yes)
