File: 4053.kicad_sch (KiCad schematic)
At the start: 3 parts, among them U3 CD4053B

Commit message: v2 initial commit
Parts:
- added R16: 100K, Resistor_THT:R_Axial_DIN0207_L6.3mm_D2.5mm_P10.16mm_Horizontal, symbol Device:R_Small
- renumbered R2 to R17, R1 to R18, U3 to U7
Connections:
- net GND: now also R16.2
- net Select: no longer U7.9 (S3)
- new net S3: R16.1, U7.9 (S3)
Other:
- moved on the sheet: R17

Commit message: schematic finished
Parts:
- renumbered R17 to R19, R16 to R20, R18 to R21, U7 to U5
Changed lines of the file:
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@@
 		(dnp no)
 		(fields_autoplaced yes)
-		(property "Reference" "#PWR026"
+		(property "Reference" "#PWR032"
 			(at 111.76 120.65 0)
 			(effects
@@
 			(project "kleingorium"
 				(path "/01c1f2c1-4d06-4880-847a-9ab55552e3fd/ad1f1d92-237d-4bc3-883c-2ce266dd223f/247fb682-d730-405d-8497-89081ac41489"
-					(reference "#PWR026")
+					(reference "#PWR032")
+					(unit 1)
+				)
+				(path "/01c1f2c1-4d06-4880-847a-9ab55552e3fd/ad1f1d92-237d-4bc3-883c-2ce266dd223f/d800d029-a2d1-4bc5-93d8-cd4a96c632ef"
+					(reference "#PWR052")
 					(unit 1)
 				)
@@
 		(dnp no)
 		(fields_autoplaced yes)
-		(property "Reference" "#PWR027"
+		(property "Reference" "#PWR031"
 			(at 102.87 120.65 0)
 			(effects
@@
 			(project "kleingorium"
 				(path "/01c1f2c1-4d06-4880-847a-9ab55552e3fd/ad1f1d92-237d-4bc3-883c-2ce266dd223f/247fb682-d730-405d-8497-89081ac41489"
-					(reference "#PWR027")
+					(reference "#PWR031")
+					(unit 1)
+				)
+				(path "/01c1f2c1-4d06-4880-847a-9ab55552e3fd/ad1f1d92-237d-4bc3-883c-2ce266dd223f/d800d029-a2d1-4bc5-93d8-cd4a96c632ef"
+					(reference "#PWR051")
 					(unit 1)
 				)
@@
 					(unit 1)
 				)
+				(path "/01c1f2c1-4d06-4880-847a-9ab55552e3fd/ad1f1d92-237d-4bc3-883c-2ce266dd223f/d800d029-a2d1-4bc5-93d8-cd4a96c632ef"
+					(reference "#PWR053")
+					(unit 1)
+				)
 			)
 		)
@@
 		(on_board yes)
 		(dnp no)
-		(property "Reference" "R16"
+		(property "Reference" "R20"
 			(at 105.664 104.14 0)
 			(effects
@@
 			(project "kleingorium"
 				(path "/01c1f2c1-4d06-4880-847a-9ab55552e3fd/ad1f1d92-237d-4bc3-883c-2ce266dd223f/247fb682-d730-405d-8497-89081ac41489"
-					(reference "R16")
+					(reference "R20")
+					(unit 1)
+				)
+				(path "/01c1f2c1-4d06-4880-847a-9ab55552e3fd/ad1f1d92-237d-4bc3-883c-2ce266dd223f/d800d029-a2d1-4bc5-93d8-cd4a96c632ef"
+					(reference "R31")
 					(unit 1)
 				)
@@
 		(dnp no)
 		(fields_autoplaced yes)
-		(property "Reference" "R18"
+		(property "Reference" "R21"
 			(at 124.46 104.1399 0)
 			(effects
@@
 			(project "kleingorium"
 				(path "/01c1f2c1-4d06-4880-847a-9ab55552e3fd/ad1f1d92-237d-4bc3-883c-2ce266dd223f/247fb682-d730-405d-8497-89081ac41489"
-					(reference "R18")
+					(reference "R21")
+					(unit 1)
+				)
+				(path "/01c1f2c1-4d06-4880-847a-9ab55552e3fd/ad1f1d92-237d-4bc3-883c-2ce266dd223f/d800d029-a2d1-4bc5-93d8-cd4a96c632ef"
+					(reference "R32")
 					(unit 1)
 				)
@@
 					(unit 1)
 				)
+				(path "/01c1f2c1-4d06-4880-847a-9ab55552e3fd/ad1f1d92-237d-4bc3-883c-2ce266dd223f/d800d029-a2d1-4bc5-93d8-cd4a96c632ef"
+					(reference "#PWR054")
+					(unit 1)
+				)
 			)
 		)
@@
 		(dnp no)
 		(fields_autoplaced yes)
-		(property "Reference" "U7"
+		(property "Reference" "U5"
 			(at 139.3033 60.96 0)
 			(effects
@@
 			(project "kleingorium"
 				(path "/01c1f2c1-4d06-4880-847a-9ab55552e3fd/ad1f1d92-237d-4bc3-883c-2ce266dd223f/247fb682-d730-405d-8497-89081ac41489"
-					(reference "U7")
+					(reference "U5")
+					(unit 1)
+				)
+				(path "/01c1f2c1-4d06-4880-847a-9ab55552e3fd/ad1f1d92-237d-4bc3-883c-2ce266dd223f/d800d029-a2d1-4bc5-93d8-cd4a96c632ef"
+					(reference "U9")
 					(unit 1)
 				)
@@
 					(unit 1)
 				)
+				(path "/01c1f2c1-4d06-4880-847a-9ab55552e3fd/ad1f1d92-237d-4bc3-883c-2ce266dd223f/d800d029-a2d1-4bc5-93d8-cd4a96c632ef"
+					(reference "#PWR056")
+					(unit 1)
+				)
 			)
 		)
@@
 					(unit 1)
 				)
+				(path "/01c1f2c1-4d06-4880-847a-9ab55552e3fd/ad1f1d92-237d-4bc3-883c-2ce266dd223f/d800d029-a2d1-4bc5-93d8-cd4a96c632ef"
+					(reference "#PWR055")
+					(unit 1)
+				)
 			)
 		)
@@
 		(on_board yes)
 		(dnp no)
-		(property "Reference" "R17"
+		(property "Reference" "R19"
 			(at 96.012 104.14 0)
 			(effects
@@
 			(project "kleingorium"
 				(path "/01c1f2c1-4d06-4880-847a-9ab55552e3fd/ad1f1d92-237d-4bc3-883c-2ce266dd223f/247fb682-d730-405d-8497-89081ac41489"
-					(reference "R17")
-					(unit 1)
-				)
+					(reference "R19")
+					(unit 1)
+				)
+				(path "/01c1f2c1-4d06-4880-847a-9ab55552e3fd/ad1f1d92-237d-4bc3-883c-2ce266dd223f/d800d029-a2d1-4bc5-93d8-cd4a96c632ef"
+					(reference "R30")
+					(unit 1)
+				)

Commit message: wip symmetric layout
Parts:
- renumbered R19 to R20, R20 to R21, R21 to R22, U5 to U6
Changed lines of the file:
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@@
 		(dnp no)
 		(fields_autoplaced yes)
-		(property "Reference" "#PWR032"
+		(property "Reference" "#PWR034"
 			(at 111.76 120.65 0)
 			(effects
@@
 		(instances
 			(project "kleingorium"
-				(path "/01c1f2c1-4d06-4880-847a-9ab55552e3fd/ad1f1d92-237d-4bc3-883c-2ce266dd223f/247fb682-d730-405d-8497-89081ac41489"
-					(reference "#PWR032")
-					(unit 1)
-				)
-				(path "/01c1f2c1-4d06-4880-847a-9ab55552e3fd/ad1f1d92-237d-4bc3-883c-2ce266dd223f/d800d029-a2d1-4bc5-93d8-cd4a96c632ef"
-					(reference "#PWR052")
+				(path "/01c1f2c1-4d06-4880-847a-9ab55552e3fd/ad1f1d92-237d-4bc3-883c-2ce266dd223f/4b203833-f0af-4e88-a9fb-191df5175df3/e87654c9-828e-47c8-8517-1d68e188f7a7"
+					(reference "#PWR020")
+					(unit 1)
+				)
+				(path "/01c1f2c1-4d06-4880-847a-9ab55552e3fd/ad1f1d92-237d-4bc3-883c-2ce266dd223f/e00ebc01-440e-4477-8d51-aed2c51c95ea/e87654c9-828e-47c8-8517-1d68e188f7a7"
+					(reference "#PWR034")
 					(unit 1)
 				)
@@
 		(dnp no)
 		(fields_autoplaced yes)
-		(property "Reference" "#PWR031"
+		(property "Reference" "#PWR033"
 			(at 102.87 120.65 0)
 			(effects
@@
 		(instances
 			(project "kleingorium"
-				(path "/01c1f2c1-4d06-4880-847a-9ab55552e3fd/ad1f1d92-237d-4bc3-883c-2ce266dd223f/247fb682-d730-405d-8497-89081ac41489"
-					(reference "#PWR031")
-					(unit 1)
-				)
-				(path "/01c1f2c1-4d06-4880-847a-9ab55552e3fd/ad1f1d92-237d-4bc3-883c-2ce266dd223f/d800d029-a2d1-4bc5-93d8-cd4a96c632ef"
-					(reference "#PWR051")
+				(path "/01c1f2c1-4d06-4880-847a-9ab55552e3fd/ad1f1d92-237d-4bc3-883c-2ce266dd223f/4b203833-f0af-4e88-a9fb-191df5175df3/e87654c9-828e-47c8-8517-1d68e188f7a7"
+					(reference "#PWR019")
+					(unit 1)
+				)
+				(path "/01c1f2c1-4d06-4880-847a-9ab55552e3fd/ad1f1d92-237d-4bc3-883c-2ce266dd223f/e00ebc01-440e-4477-8d51-aed2c51c95ea/e87654c9-828e-47c8-8517-1d68e188f7a7"
+					(reference "#PWR033")
 					(unit 1)
 				)
@@
 		(on_board yes)
 		(dnp no)
-		(property "Reference" "#PWR033"
+		(property "Reference" "#PWR035"
 			(at 121.92 120.65 0)
 			(effects
@@
 		(instances
 			(project "kleingorium"
-				(path "/01c1f2c1-4d06-4880-847a-9ab55552e3fd/ad1f1d92-237d-4bc3-883c-2ce266dd223f/247fb682-d730-405d-8497-89081ac41489"
-					(reference "#PWR033")
-					(unit 1)
-				)
-				(path "/01c1f2c1-4d06-4880-847a-9ab55552e3fd/ad1f1d92-237d-4bc3-883c-2ce266dd223f/d800d029-a2d1-4bc5-93d8-cd4a96c632ef"
-					(reference "#PWR053")
+				(path "/01c1f2c1-4d06-4880-847a-9ab55552e3fd/ad1f1d92-237d-4bc3-883c-2ce266dd223f/4b203833-f0af-4e88-a9fb-191df5175df3/e87654c9-828e-47c8-8517-1d68e188f7a7"
+					(reference "#PWR021")
+					(unit 1)
+				)
+				(path "/01c1f2c1-4d06-4880-847a-9ab55552e3fd/ad1f1d92-237d-4bc3-883c-2ce266dd223f/e00ebc01-440e-4477-8d51-aed2c51c95ea/e87654c9-828e-47c8-8517-1d68e188f7a7"
+					(reference "#PWR035")
 					(unit 1)
 				)
@@
 		(on_board yes)
 		(dnp no)
-		(property "Reference" "R20"
+		(property "Reference" "R21"
 			(at 105.664 104.14 0)
 			(effects
@@
 		(instances
 			(project "kleingorium"
-				(path "/01c1f2c1-4d06-4880-847a-9ab55552e3fd/ad1f1d92-237d-4bc3-883c-2ce266dd223f/247fb682-d730-405d-8497-89081ac41489"
-					(reference "R20")
-					(unit 1)
-				)
-				(path "/01c1f2c1-4d06-4880-847a-9ab55552e3fd/ad1f1d92-237d-4bc3-883c-2ce266dd223f/d800d029-a2d1-4bc5-93d8-cd4a96c632ef"
-					(reference "R31")
+				(path "/01c1f2c1-4d06-4880-847a-9ab55552e3fd/ad1f1d92-237d-4bc3-883c-2ce266dd223f/4b203833-f0af-4e88-a9fb-191df5175df3/e87654c9-828e-47c8-8517-1d68e188f7a7"
+					(reference "R12")
+					(unit 1)
+				)
+				(path "/01c1f2c1-4d06-4880-847a-9ab55552e3fd/ad1f1d92-237d-4bc3-883c-2ce266dd223f/e00ebc01-440e-4477-8d51-aed2c51c95ea/e87654c9-828e-47c8-8517-1d68e188f7a7"
+					(reference "R21")
 					(unit 1)
 				)
@@
 		(dnp no)
 		(fields_autoplaced yes)
-		(property "Reference" "R21"
+		(property "Reference" "R22"
 			(at 124.46 104.1399 0)
 			(effects
@@
 		(instances
 			(project "kleingorium"
-				(path "/01c1f2c1-4d06-4880-847a-9ab55552e3fd/ad1f1d92-237d-4bc3-883c-2ce266dd223f/247fb682-d730-405d-8497-89081ac41489"
-					(reference "R21")
-					(unit 1)
-				)
-				(path "/01c1f2c1-4d06-4880-847a-9ab55552e3fd/ad1f1d92-237d-4bc3-883c-2ce266dd223f/d800d029-a2d1-4bc5-93d8-cd4a96c632ef"
-					(reference "R32")
+				(path "/01c1f2c1-4d06-4880-847a-9ab55552e3fd/ad1f1d92-237d-4bc3-883c-2ce266dd223f/4b203833-f0af-4e88-a9fb-191df5175df3/e87654c9-828e-47c8-8517-1d68e188f7a7"
+					(reference "R19")
+					(unit 1)
+				)
+				(path "/01c1f2c1-4d06-4880-847a-9ab55552e3fd/ad1f1d92-237d-4bc3-883c-2ce266dd223f/e00ebc01-440e-4477-8d51-aed2c51c95ea/e87654c9-828e-47c8-8517-1d68e188f7a7"
+					(reference "R22")
 					(unit 1)
 				)
@@
 		(dnp no)
 		(fields_autoplaced yes)
-		(property "Reference" "#PWR034"
+		(property "Reference" "#PWR036"
 			(at 129.54 120.65 0)
 			(effects
@@
 		(instances
 			(project "kleingorium"
-				(path "/01c1f2c1-4d06-4880-847a-9ab55552e3fd/ad1f1d92-237d-4bc3-883c-2ce266dd223f/247fb682-d730-405d-8497-89081ac41489"
-					(reference "#PWR034")
-					(unit 1)
-				)
-				(path "/01c1f2c1-4d06-4880-847a-9ab55552e3fd/ad1f1d92-237d-4bc3-883c-2ce266dd223f/d800d029-a2d1-4bc5-93d8-cd4a96c632ef"
-					(reference "#PWR054")
+				(path "/01c1f2c1-4d06-4880-847a-9ab55552e3fd/ad1f1d92-237d-4bc3-883c-2ce266dd223f/4b203833-f0af-4e88-a9fb-191df5175df3/e87654c9-828e-47c8-8517-1d68e188f7a7"
+					(reference "#PWR022")
+					(unit 1)
+				)
+				(path "/01c1f2c1-4d06-4880-847a-9ab55552e3fd/ad1f1d92-237d-4bc3-883c-2ce266dd223f/e00ebc01-440e-4477-8d51-aed2c51c95ea/e87654c9-828e-47c8-8517-1d68e188f7a7"
+					(reference "#PWR036")
 					(unit 1)
 				)
@@
 		(dnp no)
 		(fields_autoplaced yes)
-		(property "Reference" "U5"
+		(property "Reference" "U6"
 			(at 139.3033 60.96 0)
 			(effects
@@
 		(instances
 			(project "kleingorium"
-				(path "/01c1f2c1-4d06-4880-847a-9ab55552e3fd/ad1f1d92-237d-4bc3-883c-2ce266dd223f/247fb682-d730-405d-8497-89081ac41489"
+				(path "/01c1f2c1-4d06-4880-847a-9ab55552e3fd/ad1f1d92-237d-4bc3-883c-2ce266dd223f/4b203833-f0af-4e88-a9fb-191df5175df3/e87654c9-828e-47c8-8517-1d68e188f7a7"
 					(reference "U5")
 					(unit 1)
 				)
-				(path "/01c1f2c1-4d06-4880-847a-9ab55552e3fd/ad1f1d92-237d-4bc3-883c-2ce266dd223f/d800d029-a2d1-4bc5-93d8-cd4a96c632ef"
-					(reference "U9")
+				(path "/01c1f2c1-4d06-4880-847a-9ab55552e3fd/ad1f1d92-237d-4bc3-883c-2ce266dd223f/e00ebc01-440e-4477-8d51-aed2c51c95ea/e87654c9-828e-47c8-8517-1d68e188f7a7"
+					(reference "U6")
 					(unit 1)
 				)
@@
 		(dnp no)
 		(fields_autoplaced yes)
-		(property "Reference" "#PWR036"
+		(property "Reference" "#PWR038"
 			(at 137.16 120.65 0)
 			(effects
@@
 		(instances
 			(project "kleingorium"
-				(path "/01c1f2c1-4d06-4880-847a-9ab55552e3fd/ad1f1d92-237d-4bc3-883c-2ce266dd223f/247fb682-d730-405d-8497-89081ac41489"
-					(reference "#PWR036")
-					(unit 1)
-				)
-				(path "/01c1f2c1-4d06-4880-847a-9ab55552e3fd/ad1f1d92-237d-4bc3-883c-2ce266dd223f/d800d029-a2d1-4bc5-93d8-cd4a96c632ef"
-					(reference "#PWR056")
+				(path "/01c1f2c1-4d06-4880-847a-9ab55552e3fd/ad1f1d92-237d-4bc3-883c-2ce266dd223f/4b203833-f0af-4e88-a9fb-191df5175df3/e87654c9-828e-47c8-8517-1d68e188f7a7"
+					(reference "#PWR032")
+					(unit 1)
+				)
+				(path "/01c1f2c1-4d06-4880-847a-9ab55552e3fd/ad1f1d92-237d-4bc3-883c-2ce266dd223f/e00ebc01-440e-4477-8d51-aed2c51c95ea/e87654c9-828e-47c8-8517-1d68e188f7a7"
+					(reference "#PWR038")
 					(unit 1)
 				)
@@
 		(dnp no)
 		(fields_autoplaced yes)
-		(property "Reference" "#PWR035"
+		(property "Reference" "#PWR037"
 			(at 137.16 62.23 0)
 			(effects
@@
 		(instances
 			(project "kleingorium"
-				(path "/01c1f2c1-4d06-4880-847a-9ab55552e3fd/ad1f1d92-237d-4bc3-883c-2ce266dd223f/247fb682-d730-405d-8497-89081ac41489"
-					(reference "#PWR035")
-					(unit 1)
-				)
-				(path "/01c1f2c1-4d06-4880-847a-9ab55552e3fd/ad1f1d92-237d-4bc3-883c-2ce266dd223f/d800d029-a2d1-4bc5-93d8-cd4a96c632ef"
-					(reference "#PWR055")
+				(path "/01c1f2c1-4d06-4880-847a-9ab55552e3fd/ad1f1d92-237d-4bc3-883c-2ce266dd223f/4b203833-f0af-4e88-a9fb-191df5175df3/e87654c9-828e-47c8-8517-1d68e188f7a7"
+					(reference "#PWR031")
+					(unit 1)
+				)
+				(path "/01c1f2c1-4d06-4880-847a-9ab55552e3fd/ad1f1d92-237d-4bc3-883c-2ce266dd223f/e00ebc01-440e-4477-8d51-aed2c51c95ea/e87654c9-828e-47c8-8517-1d68e188f7a7"
+					(reference "#PWR037")
 					(unit 1)
 				)
@@
 		(on_board yes)
 		(dnp no)
-		(property "Reference" "R19"
+		(property "Reference" "R20"
 			(at 96.012 104.14 0)
 			(effects
@@
 		(instances
 			(project "kleingorium"
-				(path "/01c1f2c1-4d06-4880-847a-9ab55552e3fd/ad1f1d92-237d-4bc3-883c-2ce266dd223f/247fb682-d730-405d-8497-89081ac41489"
-					(reference "R19")
-					(unit 1)
-				)
-				(path "/01c1f2c1-4d06-4880-847a-9ab55552e3fd/ad1f1d92-237d-4bc3-883c-2ce266dd223f/d800d029-a2d1-4bc5-93d8-cd4a96c632ef"
-					(reference "R30")
-					(unit 1)
-				)
+				(path "/01c1f2c1-4d06-4880-847a-9ab55552e3fd/ad1f1d92-237d-4bc3-883c-2ce266dd223f/4b203833-f0af-4e88-a9fb-191df5175df3/e87654c9-828e-47c8-8517-1d68e188f7a7"
+					(reference "R11")
+					(unit 1)
+				)
+				(path "/01c1f2c1-4d06-4880-847a-9ab55552e3fd/ad1f1d92-237d-4bc3-883c-2ce266dd223f/e00ebc01-440e-4477-8d51-aed2c51c95ea/e87654c9-828e-47c8-8517-1d68e188f7a7"
+					(reference "R20")
+					(unit 1)
+				)
