File: 4520.kicad_sch (KiCad schematic)
At the start: 7 parts, among them U4 4520

Commit message: schematic finished
Parts:
- U4: footprint (none) -> Package_DIP:DIP-16_W7.62mm
- renumbered R9 to R13, R10 to R14, R11 to R15, R12 to R16, R13 to R17, R14 to R18
Changed lines of the file:
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@@
 			)
 		)
-		(property "Footprint" ""
+		(property "Footprint" "Package_DIP:DIP-16_W7.62mm"
 			(at 38.1 36.83 0)
 			(effects
@@
 		(dnp no)
 		(fields_autoplaced yes)
-		(property "Reference" "#PWR021"
+		(property "Reference" "#PWR026"
 			(at 63.5 91.44 0)
 			(effects
@@
 			(project "kleingorium"
 				(path "/01c1f2c1-4d06-4880-847a-9ab55552e3fd/ad1f1d92-237d-4bc3-883c-2ce266dd223f/4603ebcc-7781-42ba-9745-85abd346b0eb"
-					(reference "#PWR021")
+					(reference "#PWR026")
 					(unit 1)
 				)
@@
 		(dnp no)
 		(fields_autoplaced yes)
-		(property "Reference" "R9"
+		(property "Reference" "R13"
 			(at 66.04 55.8799 0)
 			(effects
@@
 			(project "kleingorium"
 				(path "/01c1f2c1-4d06-4880-847a-9ab55552e3fd/ad1f1d92-237d-4bc3-883c-2ce266dd223f/4603ebcc-7781-42ba-9745-85abd346b0eb"
-					(reference "R9")
+					(reference "R13")
 					(unit 1)
 				)
@@
 		(dnp no)
 		(fields_autoplaced yes)
-		(property "Reference" "#PWR025"
+		(property "Reference" "#PWR030"
 			(at 87.63 96.52 0)
 			(effects
@@
 			(project "kleingorium"
 				(path "/01c1f2c1-4d06-4880-847a-9ab55552e3fd/ad1f1d92-237d-4bc3-883c-2ce266dd223f/4603ebcc-7781-42ba-9745-85abd346b0eb"
-					(reference "#PWR025")
+					(reference "#PWR030")
 					(unit 1)
 				)
@@
 		(dnp no)
 		(fields_autoplaced yes)
-		(property "Reference" "R12"
+		(property "Reference" "R16"
 			(at 78.74 83.8199 0)
 			(effects
@@
 			(project "kleingorium"
 				(path "/01c1f2c1-4d06-4880-847a-9ab55552e3fd/ad1f1d92-237d-4bc3-883c-2ce266dd223f/4603ebcc-7781-42ba-9745-85abd346b0eb"
-					(reference "R12")
+					(reference "R16")
 					(unit 1)
 				)
@@
 		(dnp no)
 		(fields_autoplaced yes)
-		(property "Reference" "#PWR018"
+		(property "Reference" "#PWR023"
 			(at 38.1 27.94 0)
 			(effects
@@
 			(project "kleingorium"
 				(path "/01c1f2c1-4d06-4880-847a-9ab55552e3fd/ad1f1d92-237d-4bc3-883c-2ce266dd223f/4603ebcc-7781-42ba-9745-85abd346b0eb"
-					(reference "#PWR018")
+					(reference "#PWR023")
 					(unit 1)
 				)
@@
 		(dnp no)
 		(fields_autoplaced yes)
-		(property "Reference" "#PWR022"
+		(property "Reference" "#PWR027"
 			(at 76.2 68.58 0)
 			(effects
@@
 			(project "kleingorium"
 				(path "/01c1f2c1-4d06-4880-847a-9ab55552e3fd/ad1f1d92-237d-4bc3-883c-2ce266dd223f/4603ebcc-7781-42ba-9745-85abd346b0eb"
-					(reference "#PWR022")
+					(reference "#PWR027")
 					(unit 1)
 				)
@@
 		(dnp no)
 		(fields_autoplaced yes)
-		(property "Reference" "R10"
+		(property "Reference" "R14"
 			(at 66.04 81.2799 0)
 			(effects
@@
 			(project "kleingorium"
 				(path "/01c1f2c1-4d06-4880-847a-9ab55552e3fd/ad1f1d92-237d-4bc3-883c-2ce266dd223f/4603ebcc-7781-42ba-9745-85abd346b0eb"
-					(reference "R10")
+					(reference "R14")
 					(unit 1)
 				)
@@
 		(dnp no)
 		(fields_autoplaced yes)
-		(property "Reference" "#PWR024"
+		(property "Reference" "#PWR029"
 			(at 87.63 71.12 0)
 			(effects
@@
 			(project "kleingorium"
 				(path "/01c1f2c1-4d06-4880-847a-9ab55552e3fd/ad1f1d92-237d-4bc3-883c-2ce266dd223f/4603ebcc-7781-42ba-9745-85abd346b0eb"
-					(reference "#PWR024")
+					(reference "#PWR029")
 					(unit 1)
 				)
@@
 		(dnp no)
 		(fields_autoplaced yes)
-		(property "Reference" "#PWR020"
+		(property "Reference" "#PWR025"
 			(at 63.5 66.04 0)
 			(effects
@@
 			(project "kleingorium"
 				(path "/01c1f2c1-4d06-4880-847a-9ab55552e3fd/ad1f1d92-237d-4bc3-883c-2ce266dd223f/4603ebcc-7781-42ba-9745-85abd346b0eb"
-					(reference "#PWR020")
+					(reference "#PWR025")
 					(unit 1)
 				)
@@
 		(dnp no)
 		(fields_autoplaced yes)
-		(property "Reference" "#PWR019"
+		(property "Reference" "#PWR024"
 			(at 38.1 55.88 0)
 			(effects
@@
 			(project "kleingorium"
 				(path "/01c1f2c1-4d06-4880-847a-9ab55552e3fd/ad1f1d92-237d-4bc3-883c-2ce266dd223f/4603ebcc-7781-42ba-9745-85abd346b0eb"
-					(reference "#PWR019")
+					(reference "#PWR024")
 					(unit 1)
 				)
@@
 		(dnp no)
 		(fields_autoplaced yes)
-		(property "Reference" "R11"
+		(property "Reference" "R15"
 			(at 78.74 58.4199 0)
 			(effects
@@
 			(project "kleingorium"
 				(path "/01c1f2c1-4d06-4880-847a-9ab55552e3fd/ad1f1d92-237d-4bc3-883c-2ce266dd223f/4603ebcc-7781-42ba-9745-85abd346b0eb"
-					(reference "R11")
+					(reference "R15")
 					(unit 1)
 				)
@@
 			)
 		)
-		(property "Footprint" ""
+		(property "Footprint" "Package_DIP:DIP-16_W7.62mm"
 			(at 100.33 80.01 0)
 			(effects
@@
 		(dnp no)
 		(fields_autoplaced yes)
-		(property "Reference" "#PWR023"
+		(property "Reference" "#PWR028"
 			(at 76.2 93.98 0)
 			(effects
@@
 			(project "kleingorium"
 				(path "/01c1f2c1-4d06-4880-847a-9ab55552e3fd/ad1f1d92-237d-4bc3-883c-2ce266dd223f/4603ebcc-7781-42ba-9745-85abd346b0eb"
-					(reference "#PWR023")
+					(reference "#PWR028")
 					(unit 1)
 				)
@@
 		(dnp no)
 		(fields_autoplaced yes)
-		(property "Reference" "R14"
+		(property "Reference" "R18"
 			(at 90.17 86.3599 0)
 			(effects
@@
 			(project "kleingorium"
 				(path "/01c1f2c1-4d06-4880-847a-9ab55552e3fd/ad1f1d92-237d-4bc3-883c-2ce266dd223f/4603ebcc-7781-42ba-9745-85abd346b0eb"
-					(reference "R14")
+					(reference "R18")
 					(unit 1)
 				)
@@
 			)
 		)
-		(property "Footprint" ""
+		(property "Footprint" "Package_DIP:DIP-16_W7.62mm"
 			(at 100.33 54.61 0)
 			(effects
@@
 		(dnp no)
 		(fields_autoplaced yes)
-		(property "Reference" "R13"
+		(property "Reference" "R17"
 			(at 90.17 60.9599 0)
 			(effects
@@
 			(project "kleingorium"
 				(path "/01c1f2c1-4d06-4880-847a-9ab55552e3fd/ad1f1d92-237d-4bc3-883c-2ce266dd223f/4603ebcc-7781-42ba-9745-85abd346b0eb"
-					(reference "R13")
-					(unit 1)
-				)
+					(reference "R17")
+					(unit 1)
+				)

Commit message: two halves routing
Parts:
- removed R13, R14: 100K, Resistor_THT:R_Axial_DIN0207_L6.3mm_D2.5mm_P10.16mm_Horizontal, symbol Device:R_Small
