File: 4520.kicad_sch (KiCad schematic)
At the start: 5 parts, among them U4 4520

Commit message: start smd refactoring
Parts:
- R15, R16, R17, R18: footprint Resistor_THT:R_Axial_DIN0207_L6.3mm_D2.5mm_P10.16mm_Horizontal -> R_0805_2012Metric; KiLib_Generator (none) -> SMD_2terminal_chip_molded
- U4: footprint Package_DIP:DIP-16_W7.62mm -> SOIC-16_3.9x9.9mm_P1.27mm; KiLib_Generator (none) -> package/gullwing
Changed lines of the file:
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@@
 			)
 		)
-		(property "Footprint" "Package_DIP:DIP-16_W7.62mm"
+		(property "Footprint" "SOIC-16_3.9x9.9mm_P1.27mm"
 			(at 38.1 36.83 0)
 			(hide yes)
@@
 			)
 		)
-		(property "Datasheet" "http://www.intersil.com/content/dam/Intersil/documents/cd45/cd4518bms-20bms.pdf"
+		(property "Datasheet" ""
 			(at 38.1 36.83 0)
 			(hide yes)
@@
 			)
 		)
-		(property "Description" "Dual Binary Up-Counter"
+		(property "Description" ""
+			(at 38.1 36.83 0)
+			(hide yes)
+			(show_name no)
+			(do_not_autoplace no)
+			(effects
+				(font
+					(size 1.27 1.27)
+				)
+			)
+		)
+		(property "KiLib_Generator" "package/gullwing"
 			(at 38.1 36.83 0)
 			(hide yes)
@@
 			)
 		)
-		(property "Footprint" "Resistor_THT:R_Axial_DIN0207_L6.3mm_D2.5mm_P10.16mm_Horizontal"
+		(property "Footprint" "R_0805_2012Metric"
 			(at 76.2 85.09 0)
 			(hide yes)
@@
 			)
 		)
-		(property "Description" "Resistor, small symbol"
+		(property "Description" ""
+			(at 76.2 85.09 0)
+			(hide yes)
+			(show_name no)
+			(do_not_autoplace no)
+			(effects
+				(font
+					(size 1.27 1.27)
+				)
+			)
+		)
+		(property "KiLib_Generator" "SMD_2terminal_chip_molded"
 			(at 76.2 85.09 0)
 			(hide yes)
@@
 			)
 		)
-		(property "Footprint" "Resistor_THT:R_Axial_DIN0207_L6.3mm_D2.5mm_P10.16mm_Horizontal"
+		(property "Footprint" "R_0805_2012Metric"
 			(at 76.2 59.69 0)
 			(hide yes)
@@
 			)
 		)
-		(property "Description" "Resistor, small symbol"
+		(property "Description" ""
+			(at 76.2 59.69 0)
+			(hide yes)
+			(show_name no)
+			(do_not_autoplace no)
+			(effects
+				(font
+					(size 1.27 1.27)
+				)
+			)
+		)
+		(property "KiLib_Generator" "SMD_2terminal_chip_molded"
 			(at 76.2 59.69 0)
 			(hide yes)
@@
 			)
 		)
-		(property "Footprint" "Package_DIP:DIP-16_W7.62mm"
+		(property "Footprint" "SOIC-16_3.9x9.9mm_P1.27mm"
 			(at 100.33 80.01 0)
 			(hide yes)
@@
 			)
 		)
-		(property "Datasheet" "http://www.intersil.com/content/dam/Intersil/documents/cd45/cd4518bms-20bms.pdf"
+		(property "Datasheet" ""
 			(at 100.33 80.01 0)
 			(hide yes)
@@
 			)
 		)
-		(property "Description" "Dual Binary Up-Counter"
+		(property "Description" ""
+			(at 100.33 80.01 0)
+			(hide yes)
+			(show_name no)
+			(do_not_autoplace no)
+			(effects
+				(font
+					(size 1.27 1.27)
+				)
+			)
+		)
+		(property "KiLib_Generator" "package/gullwing"
 			(at 100.33 80.01 0)
 			(hide yes)
@@
 			)
 		)
-		(property "Footprint" "Resistor_THT:R_Axial_DIN0207_L6.3mm_D2.5mm_P10.16mm_Horizontal"
+		(property "Footprint" "R_0805_2012Metric"
 			(at 87.63 87.63 0)
 			(hide yes)
@@
 			)
 		)
-		(property "Description" "Resistor, small symbol"
+		(property "Description" ""
+			(at 87.63 87.63 0)
+			(hide yes)
+			(show_name no)
+			(do_not_autoplace no)
+			(effects
+				(font
+					(size 1.27 1.27)
+				)
+			)
+		)
+		(property "KiLib_Generator" "SMD_2terminal_chip_molded"
 			(at 87.63 87.63 0)
 			(hide yes)
@@
 			)
 		)
-		(property "Footprint" "Package_DIP:DIP-16_W7.62mm"
+		(property "Footprint" "SOIC-16_3.9x9.9mm_P1.27mm"
 			(at 100.33 54.61 0)
 			(hide yes)
@@
 			)
 		)
-		(property "Datasheet" "http://www.intersil.com/content/dam/Intersil/documents/cd45/cd4518bms-20bms.pdf"
+		(property "Datasheet" ""
 			(at 100.33 54.61 0)
 			(hide yes)
@@
 			)
 		)
-		(property "Description" "Dual Binary Up-Counter"
+		(property "Description" ""
+			(at 100.33 54.61 0)
+			(hide yes)
+			(show_name no)
+			(do_not_autoplace no)
+			(effects
+				(font
+					(size 1.27 1.27)
+				)
+			)
+		)
+		(property "KiLib_Generator" "package/gullwing"
 			(at 100.33 54.61 0)
 			(hide yes)
@@
 			)
 		)
-		(property "Footprint" "Resistor_THT:R_Axial_DIN0207_L6.3mm_D2.5mm_P10.16mm_Horizontal"
+		(property "Footprint" "R_0805_2012Metric"
 			(at 87.63 62.23 0)
 			(hide yes)
@@
 			)
 		)
-		(property "Description" "Resistor, small symbol"
+		(property "Description" ""
 			(at 87.63 62.23 0)
 			(hide yes)
+			(show_name no)
+			(do_not_autoplace no)
+			(effects
+				(font
+					(size 1.27 1.27)
+				)
+			)
+		)
+		(property "KiLib_Generator" "SMD_2terminal_chip_molded"
+			(at 87.63 62.23 0)
+			(hide yes)

Commit message: clear all components, geometric constraints
Connections:
- net GND: no longer R17.2, R18.2
- net VCC: now also R17.1, R18.1
- net at U4.10 (Enable): now also R18.2; no longer R18.1
- net at U4.2 (Enable): now also R17.2; no longer R17.1
