File: multiplier_divider.kicad_sch (KiCad schematic)
At the start: 22 parts, among them J1 4017 Pins, J12 4046 Comp In, J13 Inh, J14 4053 C, J15 4053 S3, J16 4053 C0 C1, J2 4040 Output, J25 4017 Fdbk, J3 4040 Input, J4 4046 Out, J5 4046 Comp, J6 Select, J7 Output, J8 Input, J9 4046 SigIn, Q3 2N3904, Q5 2N3904, SW1 4017 Feedback, SW2 4046 CompIn, SW3 Chain

Commit message: schematic finished
Parts:
- removed J1: 4017 Pins, Connector_PinHeader_2.54mm:PinHeader_2x12_P2.54mm_Vertical, symbol Connector_Generic:Conn_02x12_Odd_Even
- added J11: Select, Connector_PinHeader_2.54mm:PinHeader_2x01_P2.54mm_Vertical, symbol Connector_Generic:Conn_02x01
- added J13: Inh, Connector_PinHeader_2.54mm:PinHeader_1x01_P2.54mm_Vertical, symbol Connector_Generic:Conn_01x01
- added J15: 4046 Comp In, Connector_PinHeader_2.54mm:PinHeader_2x01_P2.54mm_Vertical, symbol Connector_Generic:Conn_02x01
- added J17: 4046 Out, Connector_PinHeader_2.54mm:PinHeader_2x01_P2.54mm_Vertical, symbol Connector_Generic:Conn_02x01
- added J19: 4040 Input, Connector_PinHeader_2.54mm:PinHeader_1x02_P2.54mm_Vertical, symbol Connector_Generic:Conn_01x02
- added J21: 4053 S3, Connector_PinHeader_2.54mm:PinHeader_1x01_P2.54mm_Vertical, symbol Connector_Generic:Conn_01x01
- added J23: 4053 C, Connector_PinHeader_2.54mm:PinHeader_2x01_P2.54mm_Vertical, symbol Connector_Generic:Conn_02x01
- added J25: 4053 C0 C1, Connector_PinHeader_2.54mm:PinHeader_2x02_P2.54mm_Vertical, symbol Connector_Generic:Conn_02x02_Odd_Even
- added J27: 4040 Output, Connector_PinHeader_2.54mm:PinHeader_2x12_P2.54mm_Vertical, symbol Connector_Generic:Conn_02x12_Odd_Even
- added J29: 4017 Fdbk, Connector_PinHeader_2.54mm:PinHeader_2x01_P2.54mm_Vertical, symbol Connector_Generic:Conn_02x01
- added J31, J32: Output, Connector_PinHeader_2.54mm:PinHeader_2x04_P2.54mm_Vertical, symbol Connector_Generic:Conn_02x04_Odd_Even
- added J33, J34: 4017 Pins, Connector_PinSocket_2.54mm:PinSocket_2x11_P2.54mm_Vertical, symbol Connector_Generic:Conn_02x11_Odd_Even
- added J5: Input, Connector_PinHeader_2.54mm:PinHeader_2x01_P2.54mm_Vertical, symbol Connector_Generic:Conn_02x01
- added J8: 4046 SigIn, Connector_PinHeader_2.54mm:PinHeader_2x01_P2.54mm_Vertical, symbol Connector_Generic:Conn_02x01
- added Q1, Q3: 2N3904, Package_TO_SOT_THT:TO-92_Inline_Wide, symbol Transistor_BJT:2N3904
- added R1, R6: 100k, Resistor_THT:R_Axial_DIN0207_L6.3mm_D2.5mm_P10.16mm_Horizontal, symbol Device:R_Small
- added SW1: 4046 CompIn, Button_Switch_THT:SW_E-Switch_EG1271_SPDT, symbol Switch:SW_SPDT
- added SW3: 4017 Feedback, Button_Switch_THT:SW_CK_JS202011CQN_DPDT_Straight, symbol Switch:SW_DPDT_x2
- J7: value Output -> 4046 Comp
- renumbered J5 to J10, J6 to J12, J13 to J14, J12 to J16, J4 to J18, J3 to J20, J15 to J22, J14 to J24, J16 to J26, J2 to J28, J25 to J30, J8 to J6, Q5 to Q2, Q3 to Q4, R17 to R2, R15 to R7, SW1 to SW4, SW3 to SW5
Connections:
- net 4017/Q0: now also J34.1 (Pin_1); no longer SW4.1 (A)
- net 4017/Q1: now also J34.3 (Pin_3), J34.4 (Pin_4)
- net 4017/Q2: now also J34.5 (Pin_5), J34.6 (Pin_6)
- net 4017/Q3: now also J34.7 (Pin_7), J34.8 (Pin_8)
- net 4017/Q4: now also J34.10 (Pin_10), J34.9 (Pin_9)
- net 4017/Q5: now also J34.11 (Pin_11), J34.12 (Pin_12)
- net 4017/Q6: now also J34.13 (Pin_13), J34.14 (Pin_14)
- net 4017/Q7: now also J34.15 (Pin_15), J34.16 (Pin_16)
- net 4017/Q8: now also J34.17 (Pin_17), J34.18 (Pin_18)
- net 4017/Q9: now also J34.19 (Pin_19), J34.20 (Pin_20)
- net 4017/Reset: now also J34.21 (Pin_21), J34.22 (Pin_22)
- net 4520/Q1A: now also J31.1 (Pin_1), J31.2 (Pin_2)
- net 4520/Q1B: now also J32.1 (Pin_1), J32.2 (Pin_2); no longer J7.1 (Pin_1), J7.2 (Pin_2)
- net 4520/Q2A: now also J31.3 (Pin_3), J31.4 (Pin_4)
- net 4520/Q3A: now also J31.5 (Pin_5), J31.6 (Pin_6)
- net 4520/Q4A: now also J31.7 (Pin_7), J31.8 (Pin_8)
- net GND: now also R1.1, R6.1
- net VCC: now also Q1.3 (C), Q3.3 (C)
- net at SW5.1 (A): now also J5.1 (Pin_1), J5.2 (Pin_2), Q1.2 (B)
- new net: J33.22 (Pin_22), SW3.1 (A)
- new net: J34.2 (Pin_2), SW4.1 (A)
- new net: J32.3 (Pin_3), J32.4 (Pin_4)
- new net: J32.5 (Pin_5), J32.6 (Pin_6)
- new net: J32.7 (Pin_7), J32.8 (Pin_8)
- new net: J11.1 (Pin_1), J11.2 (Pin_2), Q3.2 (B)
- new net 4017 2/Clock: J17.1 (Pin_1), J17.2 (Pin_2)
- new net 4017 2/Q0: J33.21 (Pin_21)
- new net 4017 2/Q1: J33.19 (Pin_19), J33.20 (Pin_20)
- new net 4017 2/Q2: J33.17 (Pin_17), J33.18 (Pin_18)
- new net 4017 2/Q3: J33.15 (Pin_15), J33.16 (Pin_16)
- new net 4017 2/Q4: J33.13 (Pin_13), J33.14 (Pin_14)
- new net 4017 2/Q5: J33.11 (Pin_11), J33.12 (Pin_12)
- new net 4017 2/Q6: J33.10 (Pin_10), J33.9 (Pin_9)
- new net 4017 2/Q7: J33.7 (Pin_7), J33.8 (Pin_8)
- new net 4017 2/Q8: J33.5 (Pin_5), J33.6 (Pin_6)
- new net 4017 2/Q9: J33.3 (Pin_3), J33.4 (Pin_4)
- new net 4017 2/Reset: J33.1 (Pin_1), J33.2 (Pin_2), SW3.3 (C)
- new net 4040 2/Clock: J19.1 (Pin_1)
- new net 4040 2/Q0: J27.1 (Pin_1), J27.2 (Pin_2)
- new net 4040 2/Q1: J27.3 (Pin_3), J27.4 (Pin_4)
- new net 4040 2/Q10: J27.21 (Pin_21), J27.22 (Pin_22)
- new net 4040 2/Q11: J27.23 (Pin_23), J27.24 (Pin_24)
- new net 4040 2/Q2: J27.5 (Pin_5), J27.6 (Pin_6)
- new net 4040 2/Q3: J27.7 (Pin_7), J27.8 (Pin_8)
- new net 4040 2/Q4: J27.10 (Pin_10), J27.9 (Pin_9)
- new net 4040 2/Q5: J27.11 (Pin_11), J27.12 (Pin_12)
- new net 4040 2/Q6: J27.13 (Pin_13), J27.14 (Pin_14)
- new net 4040 2/Q7: J27.15 (Pin_15), J27.16 (Pin_16)
- new net 4040 2/Q8: J27.17 (Pin_17), J27.18 (Pin_18)
- new net 4040 2/Q9: J27.19 (Pin_19), J27.20 (Pin_20)
- new net 4040 2/Reset: J19.2 (Pin_2)
- new net 4046 2/Comp: J7.1 (Pin_1), J7.2 (Pin_2), SW1.2 (B)
- new net 4046 2/Inh: J13.1 (Pin_1)
- new net 4046 2/SigIn: J8.1 (Pin_1), J8.2 (Pin_2), Q1.1 (E), R1.2
- new net 4053 2/A0: J29.1 (Pin_1), J29.2 (Pin_2), SW3.2 (B)
- new net 4053 2/B: J15.1 (Pin_1), J15.2 (Pin_2), SW1.1 (A)
- new net 4053 2/C: J23.1 (Pin_1), J23.2 (Pin_2)
- new net 4053 2/C0: J25.1 (Pin_1), J25.2 (Pin_2)
- new net 4053 2/C1: J25.3 (Pin_3), J25.4 (Pin_4)
- new net 4053 2/S3: J21.1 (Pin_1)
- new net 4053 2/Select: Q3.1 (E), R6.2
Other:
- added sheet 4017 2 (4017.kicad_sch)
- added sheet 4040 2 (4040.kicad_sch)
- added sheet 4046 2 (4046.kicad_sch)
- added sheet 4053 2 (4053.kicad_sch)
- sheet 4017 ports: added none; removed Q10
- moved on the sheet: J10, J12, J14, J16, J18, J20, J22, J24, J26, J28, J30, J6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

Commit message: wip symmetric layout
Parts:
- removed J10, J7: 4046 Comp, Connector_PinHeader_2.54mm:PinHeader_2x01_P2.54mm_Vertical, symbol Connector_Generic:Conn_02x01
- removed J11, J12: Select, Connector_PinHeader_2.54mm:PinHeader_2x01_P2.54mm_Vertical, symbol Connector_Generic:Conn_02x01
- removed J13, J14: Inh, Connector_PinHeader_2.54mm:PinHeader_1x01_P2.54mm_Vertical, symbol Connector_Generic:Conn_01x01
- removed J15, J16: 4046 Comp In, Connector_PinHeader_2.54mm:PinHeader_2x01_P2.54mm_Vertical, symbol Connector_Generic:Conn_02x01
- removed J17, J18: 4046 Out, Connector_PinHeader_2.54mm:PinHeader_2x01_P2.54mm_Vertical, symbol Connector_Generic:Conn_02x01
- removed J19, J20: 4040 Input, Connector_PinHeader_2.54mm:PinHeader_1x02_P2.54mm_Vertical, symbol Connector_Generic:Conn_01x02
- removed J21, J22: 4053 S3, Connector_PinHeader_2.54mm:PinHeader_1x01_P2.54mm_Vertical, symbol Connector_Generic:Conn_01x01
- removed J23, J24: 4053 C, Connector_PinHeader_2.54mm:PinHeader_2x01_P2.54mm_Vertical, symbol Connector_Generic:Conn_02x01
- removed J25, J26: 4053 C0 C1, Connector_PinHeader_2.54mm:PinHeader_2x02_P2.54mm_Vertical, symbol Connector_Generic:Conn_02x02_Odd_Even
- removed J27, J28: 4040 Output, Connector_PinHeader_2.54mm:PinHeader_2x12_P2.54mm_Vertical, symbol Connector_Generic:Conn_02x12_Odd_Even
- removed J29, J30: 4017 Fdbk, Connector_PinHeader_2.54mm:PinHeader_2x01_P2.54mm_Vertical, symbol Connector_Generic:Conn_02x01
- removed J33, J34: 4017 Pins, Connector_PinSocket_2.54mm:PinSocket_2x11_P2.54mm_Vertical, symbol Connector_Generic:Conn_02x11_Odd_Even
- removed J5, J6: Input, Connector_PinHeader_2.54mm:PinHeader_2x01_P2.54mm_Vertical, symbol Connector_Generic:Conn_02x01
- removed J8, J9: 4046 SigIn, Connector_PinHeader_2.54mm:PinHeader_2x01_P2.54mm_Vertical, symbol Connector_Generic:Conn_02x01
- removed Q1, Q2, Q3, Q4: 2N3904, Package_TO_SOT_THT:TO-92_Inline_Wide, symbol Transistor_BJT:2N3904
- removed R1, R2, R6, R7: 100k, Resistor_THT:R_Axial_DIN0207_L6.3mm_D2.5mm_P10.16mm_Horizontal, symbol Device:R_Small
- removed SW1, SW2: 4046 CompIn, Button_Switch_THT:SW_E-Switch_EG1271_SPDT, symbol Switch:SW_SPDT
- removed SW3, SW4: 4017 Feedback, Button_Switch_THT:SW_CK_JS202011CQN_DPDT_Straight, symbol Switch:SW_DPDT_x2
Connections:
- net 4520/Q2B: now also J32.3 (Pin_3), J32.4 (Pin_4)
- net 4520/Q3B: now also J32.5 (Pin_5), J32.6 (Pin_6)
- net 4520/Q4B: now also J32.7 (Pin_7), J32.8 (Pin_8)
- net upper half/Half Input: now reaches SW5.1 (A)
Other:
- removed sheet 4017
- removed sheet 4017 2
- removed sheet 4040
- removed sheet 4040 2
- removed sheet 4046
- removed sheet 4046 2
- removed sheet 4053
- removed sheet 4053 2
- added sheet lower half (half_circuit.kicad_sch)
- added sheet upper half (half_circuit.kicad_sch)

Commit message: wip assemblying everything
Other:
- moved on the sheet: J32, SW5
