File: multiplier_divider.kicad_sch (KiCad schematic)
At the start: 3 parts, among them J31 Output, J32 Output, SW5 Chain

Commit message: start smd refactoring
Parts:
- SW5: footprint Button_Switch_THT:SW_E-Switch_EG1271_SPDT -> SW_SPDT_CK_JS102011SAQN
Changed lines of the file:
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@@
 			)
 		)
-		(property "Footprint" "Button_Switch_THT:SW_E-Switch_EG1271_SPDT"
+		(property "Footprint" "SW_SPDT_CK_JS102011SAQN"
 			(at 278.13 135.89 0)
 			(hide yes)
@@
 			)
 		)
-		(property "Description" "Switch, single pole double throw"
+		(property "Description" ""
 			(at 278.13 135.89 0)
 			(hide yes)

Commit message: back to kicad 10.0
Parts:
- SW5: footprint SW_SPDT_CK_JS102011SAQN -> Button_Switch_THT:SW_Slide_SPDT_Straight_CK_OS102011MS2Q
Changed lines of the file:
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@@
 (kicad_sch
-	(version 20260826)
+	(version 20260306)
 	(generator "eeschema")
-	(generator_version "10.99")
+	(generator_version "10.0")
 	(paper "A3")
 	(junction
@@
 			)
 		)
-		(property "Footprint" "SW_SPDT_CK_JS102011SAQN"
+		(property "Footprint" "Button_Switch_THT:SW_Slide_SPDT_Straight_CK_OS102011MS2Q"
 			(at 278.13 135.89 0)
 			(hide yes)
