File: power.kicad_sch (KiCad schematic)
At the start: 6 parts

Commit message: pcb placing doubling without routing
Parts:
- added C16, C17, C19, C20: 100nF, Capacitor_THT:C_Disc_D3.0mm_W1.6mm_P2.50mm, symbol Device:C_Small
Connections:
- net GND: now also C16.2, C17.2, C19.2, C20.2
- net VCC: now also C16.1, C17.1, C19.1, C20.1
Other:
- moved on the sheet: C10, C11, C12, C13, C14, C15

Commit message: final version v1
Parts:
- added C18: 10uF, Capacitor_THT:CP_Radial_D5.0mm_P2.50mm, symbol Device:C_Polarized
Connections:
- net GND: now also C18.2
- net VCC: now also C18.1
Changed lines of the file:
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@@
+	)
+	(junction
+		(at 110.49 87.63)
+		(diameter 0)
+		(color 0 0 0 0)
+	)
+	(junction
+		(at 110.49 74.93)
+		(diameter 0)
+		(color 0 0 0 0)
 	)
 	(junction
@@
 	(wire
 		(pts
+			(xy 110.49 74.93) (xy 118.11 74.93)
+		)
+		(stroke
+			(width 0)
+			(type default)
+		)
+	)
+	(wire
+		(pts
 			(xy 60.96 87.63) (xy 69.85 87.63)
 		)
@@
 	(wire
 		(pts
-			(xy 99.06 74.93) (xy 118.11 74.93)
+			(xy 99.06 74.93) (xy 110.49 74.93)
 		)
 		(stroke
@@
 	(wire
 		(pts
+			(xy 110.49 85.09) (xy 110.49 87.63)
+		)
+		(stroke
+			(width 0)
+			(type default)
+		)
+	)
+	(wire
+		(pts
+			(xy 110.49 87.63) (xy 118.11 87.63)
+		)
+		(stroke
+			(width 0)
+			(type default)
+		)
+	)
+	(wire
+		(pts
 			(xy 118.11 87.63) (xy 128.27 87.63)
 		)
@@
 	(wire
 		(pts
+			(xy 110.49 74.93) (xy 110.49 77.47)
+		)
+		(stroke
+			(width 0)
+			(type default)
+		)
+	)
+	(wire
+		(pts
 			(xy 60.96 74.93) (xy 69.85 74.93)
 		)
@@
 	(wire
 		(pts
-			(xy 99.06 87.63) (xy 118.11 87.63)
+			(xy 99.06 87.63) (xy 110.49 87.63)
 		)
 		(stroke
@@
 					(unit 1)
 				)
+			)
+		)
+	)
+	(symbol
+		(lib_id "Device:C_Polarized")
+		(at 110.49 81.28 0)
+		(unit 1)
+		(exclude_from_sim no)
+		(in_bom yes)
+		(on_board yes)
+		(dnp no)
+		(property "Reference" "C18"
+			(at 111.252 79.248 0)
+			(effects
+				(font
+					(size 1.27 1.27)
+				)
+				(justify left)
+			)
+		)
+		(property "Value" "10uF"
+			(at 111.76 83.566 0)
+			(effects
+				(font
+					(size 1.27 1.27)
+				)
+				(justify left)
+			)
+		)
+		(property "Footprint" "Capacitor_THT:CP_Radial_D5.0mm_P2.50mm"
+			(at 111.4552 85.09 0)
+			(effects
+				(font
+					(size 1.27 1.27)
+				)
+				(hide yes)
+			)
+		)
+		(property "Datasheet" "~"
+			(at 110.49 81.28 0)
+			(effects
+				(font
+					(size 1.27 1.27)
+				)
+				(hide yes)
+			)
+		)
+		(property "Description" "Polarized capacitor"
+			(at 110.49 81.28 0)
+			(effects
+				(font
+					(size 1.27 1.27)
+				)
+				(hide yes)
+			)
+		)
+		(pin "2"
+		)
+		(pin "1"
+		)
+		(instances
+			(project "kleingorium"
+				(path "/01c1f2c1-4d06-4880-847a-9ab55552e3fd/3ee3ba2e-f83c-4d97-8875-a2d65fcd8e09"
+					(reference "C18")
+					(unit 1)
+				)

Commit message: schematic finished
Parts:
- renumbered C13 to C10, C14 to C11, C15 to C12, C16 to C13, C17 to C14, C18 to C15, C19 to C16, C20 to C17, C10 to C7, C11 to C8, C12 to C9
