File: kleingorium.sync-conflict-20260415-011020-J4E24AU.kicad_pcb (KiCad board)
At the start: 2 copper layers, 500.1 x 100 mm, 180 parts, among them J1 VCC, J10 4046 Comp, J11 Select, J12 Select, J13 Inh, J14 Inh, J15 4046 Comp In, J16 4046 Comp In, J17 4046 Out, J18 4046 Out, J19 4040 Input, J2 VCC, J20 4040 Input, J21 4053 S3, J22 4053 S3, J23 4053 C, J24 4053 C, J25 4053 C0 C1, J26 4053 C0 C1, J27 4040 Output, J28 4040 Output, J29 4017 Fdbk, J3 GND, J30 4017 Fdbk, J31 Output, J32 Output, J33 4017 Pins, J34 4017 Pins, J35 Osc Out, J36 Conn_02x12_Odd_Even, J37 Conn_02x12_Odd_Even, J38 Conn_02x12_Odd_Even, J39 Conn_02x12_Odd_Even, J4 GND, J40 Conn_01x08, J41 Conn_01x08, J42 Osc Out, J43 Conn_02x08_Odd_Even, J44 Conn_02x08_Odd_Even, J45 Conn_02x08_Odd_Even, J46 Conn_02x08_Odd_Even, J47 Conn_02x08_Odd_Even, J48 Select, J49 Select, J5 Input, J50 Conn_02x18_Odd_Even, J51 Conn_02x18_Odd_Even, J52 Conn_02x18_Odd_Even, J53 Conn_02x18_Odd_Even, J54 Conn_02x18_Odd_Even, J55 01x18 from bottom plate, J56 VCC, J57 VCC, J58 GND, J59 GND, J6 Input, J60 VCC, J61 VCC, J62 GND, J63 GND, J64 Conn_02x08_Odd_Even, J65 Conn_02x18_Odd_Even, J66 4017 Pins, J67 4017 Pins, J68 Conn_01x16, J69 Conn_02x18_Odd_Even, J7 4046 SigIn, J70 Conn_02x18_Odd_Even, J71 Conn_02x18_Odd_Even, J72 4040 Clk Rst, J73 Conn_02x20_Odd_Even, J74 Conn_02x20_Odd_Even, J75 Conn_02x20_Odd_Even, J76 Conn_02x20_Odd_Even, J77 Conn_02x20_Odd_Even, J78 Conn_02x20_Odd_Even, J79 Conn_02x20_Odd_Even, J8 4046 Comp, J80 Conn_02x20_Odd_Even, J81 Conn_02x20_Odd_Even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

Commit message: more silkscreen, minor circuits adjustments for text
Parts:
- moved C21 175.0 mm to (603.9, 65.6), turned to 0 degrees
- moved R33 157.5 mm to (614.9, 74.5), turned to -90 degrees
- moved U11 156.0 mm to (601.1, 68.7), turned to 0 degrees
- moved U10 146.1 mm to (553.7, 71.1)
- moved C18 140.7 mm to (530.7, 88.5), turned to 0 degrees
- moved SW8 122.3 mm to (523.7, 82.2)
- moved C19 113.5 mm to (522.6, 88.7), turned to 0 degrees
- moved J72 109.4 mm to (529.0, 73.2)
- moved R19 7.23 mm to (40.5, 75.6), turned to 90 degrees
- moved RN1 2.81 mm to (477.2, 36.8)
- moved J40 2.54 mm to (472.8, 34.3)
- moved J41 2.02 mm to (492.0, 36.2)
- moved RN2 1.26 mm to (486.5, 37.3)
- moved J55 1.06 mm to (426.1, 43.4)
- moved J10 0.78 mm to (38.5, 86.7)
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Routing:
- net Net-(J87-PadT): track 216.9 -> 0.00 mm
- net GND: track 170.4 -> 16.8 mm, vias 5 -> 1
- net Net-(RN1-common): track 142.8 -> 0.00 mm
- net /Bottom plate/4051/X: track 132.5 -> 2.54 mm, vias 1 -> 0
- net Net-(RN2-common): track 110.1 -> 0.00 mm, vias 1 -> 0
- net Net-(J87-PadR): track 107.3 -> 0.00 mm
- net Net-(J35-Pin_1): track 97.6 -> 0.00 mm
- net Net-(SW8-B): track 94.6 -> 0.00 mm, vias 1 -> 0
- net VDDA: track 88.4 -> 0.00 mm
- net Net-(C18-Pad2): track 82.5 -> 0.00 mm
- net Net-(C18-Pad1): track 71.7 -> 0.00 mm
- net /Top Plate/4040/Reset: track 68.6 -> 0.00 mm
- net Net-(C19-Pad2): track 59.1 -> 0.00 mm
- net Net-(J50-Pin_7): track 50.1 -> 0.00 mm
- net Net-(J50-Pin_5): track 50.1 -> 0.00 mm
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Other:
- board text added: "𝅘𝅥𝅲 𝅘𝅥𝅱 𝅘𝅥𝅰 𝅘𝅥𝅯 𝅘𝅥𝅮 𝅘𝅥 𝅗𝅥 𝅝 𝅜 𝆷𝆶"
- board text removed: "0 1 2 3 4 5 6 7 8 9"
- board text removed: "10"
- board text removed: "11"
- board text removed: "4017 Fdbk"
- board text removed: "4046 CmpIn"
- board text removed: "4046 Out"
- board text removed: "4046 SigIn"
- board text removed: "A B C"
- board text removed: "Bottom"
- board text removed: "C1 C0"
- board text removed: "Chain"
- board text removed: "Clk"
- board text removed: "Derivative"
- board text removed: "GND"
- board text removed: "Input"
- board text removed: "Lower Output"
- board text removed: "Mult/Div"
- board text removed: "PLL Type"
- board text removed: "Proportional"
- board text removed: "Rst"
- board text removed: "Sel"
- board text removed: "Select"
- board text removed: "Upper"
- board text removed: "Upper Output"
- board text removed: "VCC"
- board text removed: "𝅜"
- board text removed: "𝅘𝅥𝅲 𝅘𝅥𝅱 𝅘𝅥𝅰 𝅘𝅥𝅯 𝅘𝅥𝅮 𝅘𝅥 𝅗𝅥 𝅝"
- board text removed: "𝆷𝆶"
