File: bottom_plate.kicad_sch (KiCad schematic)
At the start: 20 parts, among them J42 Osc Out, J43 Conn_02x08_Odd_Even, J44 Conn_02x08_Odd_Even, J45 Conn_02x08_Odd_Even, J46 Conn_02x08_Odd_Even, J47 Conn_02x08_Odd_Even, J48 Select, J49 Select, J60 VCC, J61 VCC, J62 GND, J63 GND, J64 Conn_02x08_Odd_Even, J66 4017 Pins, J67 4017 Pins, J68 Conn_02x12_Odd_Even, J73 Conn_02x12_Odd_Even, J85 Output, J86 Output, J88 Conn_01x18

Commit message: wip rerouting
Parts:
- removed J43, J44, J45, J46, J47, J64: Conn_02x08_Odd_Even, Connector_PinSocket_2.54mm:PinSocket_2x08_P2.54mm_Vertical, symbol Connector_Generic:Conn_02x08_Odd_Even
- added J74: Conn_02x09_Odd_Even, symbol Connector_Generic:Conn_02x09_Odd_Even
- added J75, J76, J77, J78, J79: Conn_02x09_Odd_Even, Connector_PinHeader_2.54mm:PinHeader_2x09_P2.54mm_Vertical, symbol Connector_Generic:Conn_02x09_Odd_Even
Connections:
- net 4051 2/A: now also J79.10 (Pin_10)
- net 4051 2/B: now also J79.12 (Pin_12)
- net 4051 2/C: now also J79.14 (Pin_14)
- net 4051 2/Inhibit: now also J68.24 (Pin_24)
- net 4051/A: now also J78.2 (Pin_2), J79.1 (Pin_1), J79.2 (Pin_2)
- net 4051/B: now also J79.4 (Pin_4)
- net 4051/C: now also J79.6 (Pin_6)
- net at J48.1 (Pin_1), J48.2 (Pin_2): now also J79.18 (Pin_18)
- net at J49.1 (Pin_1), J49.2 (Pin_2): now also J79.8 (Pin_8)
- net at J66.1 (Pin_1), J66.2 (Pin_2), J68.2 (Pin_2): now also J68.1 (Pin_1)
- net at J66.10 (Pin_10), J66.9 (Pin_9), J68.10 (Pin_10): now also J68.9 (Pin_9)
- net at J66.11 (Pin_11), J68.12 (Pin_12): now also J66.12 (Pin_12), J68.11 (Pin_11)
- net at J66.13 (Pin_13), J68.14 (Pin_14): now also J66.14 (Pin_14), J68.13 (Pin_13)
- net at J66.15 (Pin_15), J68.16 (Pin_16): now also J66.16 (Pin_16), J68.15 (Pin_15)
- net at J66.17 (Pin_17), J68.18 (Pin_18): now also J66.18 (Pin_18), J68.17 (Pin_17)
- net at J66.19 (Pin_19), J68.20 (Pin_20): now also J66.20 (Pin_20), J68.19 (Pin_19)
- net at J66.21 (Pin_21), J68.22 (Pin_22): now also J66.22 (Pin_22), J68.21 (Pin_21)
- net at J66.3 (Pin_3), J66.4 (Pin_4), J68.4 (Pin_4): now also J68.3 (Pin_3)
- net at J66.5 (Pin_5), J66.6 (Pin_6), J68.6 (Pin_6): now also J68.5 (Pin_5)
- net at J66.7 (Pin_7), J66.8 (Pin_8), J68.8 (Pin_8): now also J68.7 (Pin_7)
- new net: J77.2 (Pin_2), J78.1 (Pin_1)
- new net: J78.10 (Pin_10), J79.9 (Pin_9)
- new net: J77.12 (Pin_12), J78.11 (Pin_11)
- new net: J78.12 (Pin_12), J79.11 (Pin_11)
- new net: J77.14 (Pin_14), J78.13 (Pin_13)
- new net: J78.14 (Pin_14), J79.13 (Pin_13)
- new net: J77.16 (Pin_16), J78.15 (Pin_15)
- new net: J78.16 (Pin_16), J79.15 (Pin_15), J79.16 (Pin_16)
- new net: J77.18 (Pin_18), J78.17 (Pin_17)
- new net: J78.18 (Pin_18), J79.17 (Pin_17)
- new net: J77.4 (Pin_4), J78.3 (Pin_3)
- new net: J78.4 (Pin_4), J79.3 (Pin_3)
- new net: J77.6 (Pin_6), J78.5 (Pin_5)
- new net: J78.6 (Pin_6), J79.5 (Pin_5)
- new net: J77.8 (Pin_8), J78.7 (Pin_7)
- new net: J78.8 (Pin_8), J79.7 (Pin_7)
- new net: J77.10 (Pin_10), J78.9 (Pin_9)
- new net: J74.1 (Pin_1), J74.2 (Pin_2), J75.1 (Pin_1)
- new net: J75.10 (Pin_10), J76.9 (Pin_9)
- new net: J74.11 (Pin_11), J74.12 (Pin_12), J75.11 (Pin_11)
- new net: J75.12 (Pin_12), J76.11 (Pin_11)
- new net: J74.13 (Pin_13), J74.14 (Pin_14), J75.13 (Pin_13)
- new net: J75.14 (Pin_14), J76.13 (Pin_13)
- new net: J74.15 (Pin_15), J74.16 (Pin_16), J75.15 (Pin_15)
- new net: J75.16 (Pin_16), J76.15 (Pin_15)
- new net: J74.17 (Pin_17), J74.18 (Pin_18), J75.17 (Pin_17)
- new net: J75.18 (Pin_18), J76.17 (Pin_17)
- new net: J75.2 (Pin_2), J76.1 (Pin_1)
- new net: J74.3 (Pin_3), J74.4 (Pin_4), J75.3 (Pin_3)
- new net: J75.4 (Pin_4), J76.3 (Pin_3)
- new net: J74.5 (Pin_5), J74.6 (Pin_6), J75.5 (Pin_5)
- new net: J75.6 (Pin_6), J76.5 (Pin_5)
- new net: J74.7 (Pin_7), J74.8 (Pin_8), J75.7 (Pin_7)
- new net: J75.8 (Pin_8), J76.7 (Pin_7)
- new net: J74.10 (Pin_10), J74.9 (Pin_9), J75.9 (Pin_9)
- new net: J76.10 (Pin_10), J77.9 (Pin_9)
- new net: J76.12 (Pin_12), J77.11 (Pin_11)
- new net: J76.14 (Pin_14), J77.13 (Pin_13)
- new net: J76.16 (Pin_16), J77.15 (Pin_15)
- new net: J76.18 (Pin_18), J77.17 (Pin_17)
- new net: J76.2 (Pin_2), J77.1 (Pin_1)
- new net: J76.4 (Pin_4), J77.3 (Pin_3)
- new net: J76.6 (Pin_6), J77.5 (Pin_5)
- new net: J76.8 (Pin_8), J77.7 (Pin_7)
Other:
- added sheet 4017 (4017.kicad_sch)
- note added: "12x9 Matrix"
- note removed: "12x8 Matrix"
- moved on the sheet: J68

Commit message: top plate pin matrix
Parts:
- J74: footprint (none) -> Connector_PinHeader_2.54mm:PinHeader_2x09_P2.54mm_Vertical
Changed lines of the file:
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@@
 			)
 		)
-		(property "Footprint" ""
+		(property "Footprint" "Connector_PinHeader_2.54mm:PinHeader_2x09_P2.54mm_Vertical"
 			(at 96.52 62.23 0)
 			(hide yes)
